File: kicad/BeanBoard.kicad_sch (KiCad schematic)
At the start: 145 parts, among them SW00 SW_Push_45deg, SW01 SW_Push_45deg, SW02 SW_Push_45deg, SW03 SW_Push_45deg, SW04 SW_Push_45deg, SW05 SW_Push_45deg, SW06 SW_Push_45deg, SW07 SW_Push_45deg, SW10 SW_Push_45deg, SW11 SW_Push_45deg, SW13 SW_Push_45deg, SW14 SW_Push_45deg, SW15 SW_Push_45deg, SW16 SW_Push_45deg, SW17 SW_Push_45deg, SW20 SW_Push_45deg, SW22 SW_Push_45deg, SW23 SW_Push_45deg, SW24 SW_Push_45deg, SW25 SW_Push_45deg, SW26 SW_Push_45deg, SW27 SW_Push_45deg, SW30 SW_Push_45deg, SW31 SW_Push_45deg, SW32 SW_Push_45deg, SW33 SW_Push_45deg, SW34 SW_Push_45deg, SW37 SW_Push_45deg, SW40 SW_Push_45deg, SW41 SW_Push_45deg, SW42 SW_Push_45deg, SW43 SW_Push_45deg, SW44 SW_Push_45deg, SW45 SW_Push_45deg, SW47 SW_Push_45deg, SW50 SW_Push_45deg, SW51 SW_Push_45deg, SW52 SW_Push_45deg, SW53 SW_Push_45deg, SW54 SW_Push_45deg, SW55 SW_Push_45deg, SW56 SW_Push_45deg, SW57 SW_Push_45deg, SW60 SW_Push_45deg, SW61 SW_Push_45deg, SW62 SW_Push_45deg, SW63 SW_Push_45deg, SW64 SW_Push_45deg, SW65 SW_Push_45deg, SW66 SW_Push_45deg, SW67 SW_Push_45deg, SW70 SW_Push_45deg, SW71 SW_Push_45deg, SW72 SW_Push_45deg, SW73 SW_Push_45deg, SW74 SW_Push_45deg, SW75 SW_Push_45deg, SW76 SW_Push_45deg, SW77 SW_Push_45deg, U1 74LS32, U2 74LS04, U3 74AHCT373, U4 74LS32, U5 74LS32, U6 74LS32, U7 74LS244, U8 74LS32, U9 74LS32

Commit message: First complete pass
Parts:
- removed unit 2 of U1
- removed unit 1 of U1
- removed unit 2 of U2
- removed U6, U8, U9: 74LS32, symbol 74xx:74LS32
- added J1: BZ_Address, Connector_PinSocket_2.54mm:PinSocket_1x16_P2.54mm_Vertical, symbol Connector:Conn_01x16_Socket
- added J2: BZ_Data, Connector_PinSocket_2.54mm:PinSocket_1x08_P2.54mm_Vertical, symbol Connector:Conn_01x08_Socket
- added J3: BZ_Control, Connector_PinSocket_2.54mm:PinSocket_1x07_P2.54mm_Vertical, symbol Connector:Conn_01x07_Socket
- added J4: BZ_Power, Connector_PinSocket_2.54mm:PinSocket_1x02_P2.54mm_Vertical, symbol Connector:Conn_01x02_Socket
- added J5: BZ_IORQ_enable, Connector_PinSocket_2.54mm:PinSocket_1x07_P2.54mm_Vertical, symbol Connector:Conn_01x03_Socket
- added J6: BZ_MREQ_enable, Connector_PinSocket_2.54mm:PinSocket_1x07_P2.54mm_Vertical, symbol Connector:Conn_01x03_Socket
- added J7: LCD, Connector_PinSocket_2.54mm:PinSocket_1x16_P2.54mm_Vertical, symbol Connector:Conn_01x16_Socket
- added R9: 220R, symbol Device:R
- added RV1: 50k, symbol Device:R_Potentiometer
- added unit 3 of U2
- added U3: 74LS08, symbol 74xx:74LS08
- added U4: 74LS138, symbol 74xx:74LS138
- U5: renamed from U3; value 74AHCT373 -> SN74LS373; symbol 74xx:74AHCT373 -> 74xx:74LS373
- renumbered U5 to U1, U4 to U1, U7 to U6
Connections:
- net A0: now also J1.1 (Pin_1), U4.1 (A0); no longer U1.10
- net A1: now also J1.2 (Pin_2), U4.2 (A1); no longer U2.1
- net D0: now also J2.1 (Pin_1), J7.7 (Pin_7)
- net D1: now also J2.2 (Pin_2), J7.8 (Pin_8)
- net D2: now also J2.3 (Pin_3), J7.9 (Pin_9)
- net D3: now also J2.4 (Pin_4), J7.10 (Pin_10)
- net D4: now also J2.5 (Pin_5), J7.11 (Pin_11)
- net D5: now also J2.6 (Pin_6), J7.12 (Pin_12)
- net D6: now also J2.7 (Pin_7), J7.13 (Pin_13)
- net D7: now also J2.8 (Pin_8), J7.14 (Pin_14)
- net GND: now also U1.10, U1.12, U1.13, U1.7 (GND), U1.9, U2.11, U2.13, U2.7 (GND), U2.9, J4.2 (Pin_2), J7.1 (Pin_1), J7.16 (Pin_16), RV1.1, U2.5, U3.10, U3.12, U3.13, U3.7 (GND), U3.9, U4.8 (GND)
- net KB_WR: now also U2.4; no longer U2.6
- net VCC: now also U1.14 (VCC), U2.14 (VCC), J4.1 (Pin_1), J7.2 (Pin_2), R9.2, RV1.3, U3.14 (VCC), U4.16 (VCC)
- net ~{IORQ}: now also J3.4 (Pin_4), U4.4 (E1)
- net ~{KB_WR}: now also U2.3; no longer U2.5
- net ~{RD}: now also J3.1 (Pin_1)
- net ~{USB_IORQ}: now also J5.2 (Pin_2), U3.3
- net ~{WR}: now also J3.2 (Pin_2), J7.5 (Pin_5)
- net LCD_E: now reaches U2.2
- net LCD_E: now also J7.6 (Pin_6)
- net ~{KB_IORQ}: no longer names the net of U1.2, U1.4
- net ~{KB_IORQ}: now also U4.13 (O2); no longer U1.8
- net ~{PORT3_IORQ}: no longer names the net of U1.11
- new net: U3.5, U4.10 (O5)
- new net: U2.1, U3.6
- new net: J6.1 (Pin_1), J6.2 (Pin_2)
- new net: U3.1, U4.15 (O0)
- new net: U3.2, U4.14 (O1)
- new net A10: J1.11 (Pin_11)
- new net A11: J1.12 (Pin_12)
- new net A12: J1.13 (Pin_13)
- new net A13: J1.14 (Pin_14)
- new net A14: J1.15 (Pin_15)
- new net A15: J1.16 (Pin_16)
- new net A2: J1.3 (Pin_3), U4.3 (A2)
- new net A3: J1.4 (Pin_4)
- new net A4: J1.5 (Pin_5)
- new net A5: J1.6 (Pin_6)
- new net A6: J1.7 (Pin_7)
- new net A7: J1.8 (Pin_8)
- new net A8: J1.9 (Pin_9)
- new net A9: J1.10 (Pin_10)
- new net LCD_LED_VCC: J7.15 (Pin_15), R9.1
- new net LCD_RS: J7.4 (Pin_4), U3.4, U4.11 (O4)
- new net LCD_V0: J7.3 (Pin_3), RV1.2
- new net ~{CLKINH}: J3.7 (Pin_7)
- new net ~{CLK}: J3.6 (Pin_6)
- new net ~{MREQ}: J3.3 (Pin_3)
- new net ~{RESET}: J3.5 (Pin_5)
- no-connect marks 0 -> 6
Other:
- note added: "0 = status 1 = data"
- moved on the sheet: U1A, U1B, U1E, U2B, U2D, U2E, U2F, U2G

Commit message: Update BeanBoard.kicad_sch
Connections:
- net GND: no longer U2.5
- net ~{RD}: now also U2.5
- net ~{WR}: no longer J7.5 (Pin_5)
- net LCD_R/~{W}: now reaches U2.6
- net LCD_R/~{W}: now also J7.5 (Pin_5)
Other:
- note added: "See: https://bread80.com/2020/07/01/connecting-an-lcd-to-a-z80-with-two-glue-chips/"
- note added: "~{M1} should enable / disable IO on E3 - but we haven't made that available"
Changed lines of the file:
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@@
   (junction (at 306.07 101.6) (diameter 0) (color 0 0 0 0)
   )
-  (junction (at 90.17 266.7) (diameter 0) (color 0 0 0 0)
-  )
   (junction (at 245.11 46.99) (diameter 0) (color 0 0 0 0)
   )
@@
     (stroke (width 0) (type default))
   )
+  (wire (pts (xy 41.91 96.52) (xy 46.99 96.52))
+    (stroke (width 0) (type default))
+  )
   (wire (pts (xy 123.19 168.91) (xy 123.19 171.45))
     (stroke (width 0) (type default))
@@
     (stroke (width 0) (type default))
   )
-  (wire (pts (xy 90.17 251.46) (xy 90.17 266.7))
-    (stroke (width 0) (type default))
-  )
   (wire (pts (xy 104.14 62.23) (xy 96.52 62.23))
     (stroke (width 0) (type default))
@@
     (stroke (width 0) (type default))
   )
+  (wire (pts (xy 62.23 96.52) (xy 73.66 96.52))
+    (stroke (width 0) (type default))
+  )
   (wire (pts (xy 295.91 31.75) (xy 295.91 46.99))
     (stroke (width 0) (type default))
@@
     (stroke (width 0) (type default))
   )
+  (text "~{M1} should enable / disable IO on E3\n- but we haven't made that available"
+    (at 15.24 36.83 0)
+    (effects (font (size 1.27 1.27)) (justify left bottom))
+  )
+  (text "See: https://bread80.com/2020/07/01/connecting-an-lcd-to-a-z80-with-two-glue-chips/\n"
+    (at 41.91 104.14 0)
+    (effects (font (size 1.27 1.27)) (justify left bottom))
+  )
   (text "0 = status\n1 = data" (at 78.74 60.96 0)
     (effects (font (size 1.27 1.27)) (justify left bottom))
@@
     (effects (font (size 1.27 1.27)) (justify left bottom))
   )
+  (label "~{RD}" (at 41.91 96.52 0) (fields_autoplaced)
+    (effects (font (size 1.27 1.27)) (justify left bottom))
+  )
   (label "D4" (at 54.61 128.27 180) (fields_autoplaced)
     (effects (font (size 1.27 1.27)) (justify right bottom))
@@
     (effects (font (size 1.27 1.27)) (justify right bottom))
   )
-  (label "~{KB_RD}" (at 349.25 101.6 0) (fields_autoplaced)
-    (effects (font (size 1.27 1.27)) (justify left bottom))
+  (label "LCD_R{slash}~{W}" (at 73.66 96.52 180) (fields_autoplaced)
+    (effects (font (size 1.27 1.27)) (justify right bottom))
   )
-  (label "~{WR}" (at 125.73 129.54 0) (fields_autoplaced)
+  (label "~{KB_RD}" (at 349.25 101.6 0) (fields_autoplaced)
     (effects (font (size 1.27 1.27)) (justify left bottom))
   )
@@
     (effects (font (size 1.27 1.27)) (justify left bottom))
   )
+  (label "LCD_R{slash}~{W}" (at 125.73 129.54 0) (fields_autoplaced)
+    (effects (font (size 1.27 1.27)) (justify left bottom))
+  )
   (symbol (lib_id "Switch:SW_Push") (at 237.49 93.98 0) (unit 1)
     (in_bom yes) (on_board yes) (dnp no) (fields_autoplaced)
@@
     )
   )
+  (symbol (lib_id "74xx:74LS04") (at 54.61 96.52 0) (unit 3)
+    (in_bom yes) (on_board yes) (dnp no) (fields_autoplaced)
+    (property "Reference" "U2" (at 54.61 87.63 0)
+      (effects (font (size 1.27 1.27)))
+    )
+    (property "Value" "74LS04" (at 54.61 90.17 0)
+      (effects (font (size 1.27 1.27)))
+    )
+    (property "Footprint" "" (at 54.61 96.52 0)
+      (effects (font (size 1.27 1.27)) hide)
+    )
+    (property "Datasheet" "http://www.ti.com/lit/gpn/sn74LS04" (at 54.61 96.52 0)
+      (effects (font (size 1.27 1.27)) hide)
+    )
+    (pin "10")
+    (pin "14")
+    (pin "7")
+    (pin "6")
+    (pin "8")
+    (pin "9")
+    (pin "5")
+    (pin "12")
+    (pin "2")
+    (pin "13")
+    (pin "3")
+    (pin "4")
+    (pin "1")
+    (pin "11")
+    (instances
+      (project "BeanBoard"
+        (path "/3defbfd6-25f4-40d7-986c-89ce878d27b9"
+          (reference "U2") (unit 3)
+        )
+      )
+    )
+  )
   (symbol (lib_id "Device:R") (at 223.52 101.6 90) (unit 1)
     (in_bom yes) (on_board yes) (dnp no) (fields_autoplaced)
@@
         )
       )
-    )
-  )
-  (symbol (lib_id "74xx:74LS04") (at 97.79 251.46 0) (unit 3)
-    (in_bom yes) (on_board yes) (dnp no) (fields_autoplaced)
-    (property "Reference" "U2" (at 97.79 242.57 0)
-      (effects (font (size 1.27 1.27)))
-    )
-    (property "Value" "74LS04" (at 97.79 245.11 0)
-      (effects (font (size 1.27 1.27)))
-    )
-    (property "Footprint" "" (at 97.79 251.46 0)
-      (effects (font (size 1.27 1.27)) hide)
-    )
-    (property "Datasheet" "http://www.ti.com/lit/gpn/sn74LS04" (at 97.79 251.46 0)
-      (effects (font (size 1.27 1.27)) hide)
-    )
-    (pin "10")
-    (pin "14")
-    (pin "7")
-    (pin "6")
-    (pin "8")
-    (pin "9")
-    (pin "5")
-    (pin "12")
-    (pin "2")
-    (pin "13")
-    (pin "3")
-    (pin "4")
-    (pin "1")
-    (pin "11")
-    (instances
-      (project "BeanBoard"
-        (path "/3defbfd6-25f4-40d7-986c-89ce878d27b9"
-          (reference "U2") (unit 3)
-        )
-      )

Commit message: Update BeanBoard.kicad_sch
Parts:
- removed U3: 74LS08, symbol 74xx:74LS08
Connections:
- net A0: now also J7.4 (Pin_4); no longer U4.1 (A0)
- net A1: now also U4.1 (A0); no longer U4.2 (A1)
- net A2: now also U4.2 (A1); no longer U4.3 (A2)
- net A3: now also U4.3 (A2)
- net GND: now also U4.4 (E1)
- net VCC: now also U4.6 (E3)
- net ~{IORQ}: now also U4.5 (E2); no longer U4.4 (E1)
- net ~{USB_IORQ}: now also U4.15 (O0)
- net ~{KB_E}: now reaches U1.2, U1.4
- net ~{KB_E}: now also U4.14 (O1); no longer U4.13 (O2)
- net ~{LCD_E}: now reaches U2.1
- net ~{LCD_E}: now also U4.13 (O2)
- net LCD_RS: no longer names the net of U4.11 (O4)
- net LCD_RS: no longer J7.4 (Pin_4)
- no-connect marks 6 -> 13
Other:
- note added: "~{M1} should enable / disable IO on E3 - but we haven't made that available on BeanZee"
- note removed: "~{M1} should enable / disable IO on E3 - but we haven't made that available"
- moved on the sheet: J1, J2, J3, J4, J5, J6, J7, R1, R2, R3, R4, R5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

Commit message: Update BeanBoard.kicad_sch
Parts:
- added C1, C2, C3, C4, C5: 0.1uF, Capacitor_THT:C_Disc_D5.0mm_W2.5mm_P2.50mm, symbol Device:C
- R1, R2, R3, R4, R5, R6, R7, R8, R9: footprint (none) -> Resistor_THT:R_Axial_DIN0204_L3.6mm_D1.6mm_P7.62mm_Horizontal
Connections:
- net GND: now also C1.1, C2.1, C3.1, C4.2, C5.2
- net VCC: now also C1.2, C2.2, C3.2, C4.1, C5.1
- no-connect marks 13 -> 29
Other:
- note added: "LCD GND"
- note added: "LCD VCC"
- note added: "LCD_RS"
- note added: "LED"
- note removed: "See: https://bread80.com/2020/07/01/connecting-an-lcd-to-a-z80-with-two-glue-chips/"
- moved on the sheet: J4, U2C

Commit message: Update BeanBoard.kicad_sch
Parts:
- RV1: footprint (none) -> Connector_PinSocket_2.54mm:PinSocket_1x03_P2.54mm_Vertical
- S12, S21, SW00, SW01, SW02, SW03, SW04, SW05, SW06, SW07, SW10, SW11, SW13, SW14, SW15, SW16, SW17, SW20, SW22, SW23, SW24, SW25, SW26, SW27, SW30, SW31, SW32, SW33, SW34, SW37, SW40, SW41, SW42, SW43, SW44, SW45, SW47, SW50, SW51, SW52, SW53, SW54, SW55, SW56, SW57, SW60, SW61, SW62, SW63, SW64, SW65, SW66, SW67, SW70, SW71, SW72, SW73, SW74, SW75, SW76, SW77, SWC46, SWD35, SWX36: footprint (none) -> SW_B3F-4000_OMR:SW_B3F-4000_OMR
- U1, U2: footprint (none) -> Package_DIP:DIP-14_W7.62mm_Socket_LongPads
- U4: footprint (none) -> Package_DIP:DIP-16_W7.62mm_Socket_LongPads
- U5, U6: footprint (none) -> Package_DIP:DIP-20_W7.62mm_Socket_LongPads

Commit message: Update BeanBoard.kicad_sch
Parts:
- RV1: footprint Connector_PinSocket_2.54mm:PinSocket_1x03_P2.54mm_Vertical -> (none)
- S12, S21, SW00, SW01, SW02, SW03, SW04, SW05, SW06, SW07, SW10, SW11, SW13, SW14, SW15, SW16, SW17, SW20, SW22, SW23, SW24, SW25, SW26, SW27, SW30, SW31, SW32, SW33, SW34, SW37, SW40, SW41, SW42, SW43, SW44, SW45, SW47, SW50, SW51, SW52, SW53, SW54, SW55, SW56, SW57, SW60, SW61, SW62, SW63, SW64, SW65, SW66, SW67, SW70, SW71, SW72, SW73, SW74, SW75, SW76, SW77, SWC46, SWD35, SWX36: footprint SW_B3F-4000_OMR:SW_B3F-4000_OMR -> (none)

Commit message: Update BeanBoard.kicad_sch
Parts:
- removed unit 3 of U1
- removed unit 4 of U1
- removed unit 4 of U2
- added C6, C7: 0.1uF, Capacitor_THT:C_Disc_D5.0mm_W2.5mm_P2.50mm, symbol Device:C
- added J8: GPO, Connector_PinSocket_2.54mm:PinSocket_1x08_P2.54mm_Vertical, symbol Connector:Conn_01x08_Socket
- added J9: GPI, Connector_PinSocket_2.54mm:PinSocket_1x08_P2.54mm_Vertical, symbol Connector:Conn_01x08_Socket
- added U4: SN74LS373, Package_DIP:DIP-20_W7.62mm_Socket_LongPads, symbol 74xx:74LS373
- added U5: 74LS244, Package_DIP:DIP-20_W7.62mm_Socket_LongPads, symbol 74xx:74LS244
- added unit 4 of U6
- added unit 3 of U6
- added unit 4 of U7
- RV1: footprint (none) -> Connector_PinSocket_2.54mm:PinSocket_1x03_P2.54mm_Vertical
- SW00, SW01, SW02, SW03, SW04, SW05, SW06, SW07, SW10, SW11, SW13, SW14, SW15, SW16, SW17, SW20, SW22, SW23, SW24, SW25, SW26, SW27, SW30, SW31, SW32, SW33, SW34, SW37, SW40, SW41, SW42, SW43, SW44, SW45, SW47, SW50, SW51, SW52, SW53, SW54, SW55, SW56, SW57, SW60, SW61, SW62, SW63, SW64, SW65, SW66, SW67, SW70, SW71, SW72, SW73, SW74, SW75, SW76, SW77: footprint (none) -> SW_B3F-4000_OMR:SW_B3F-4000_OMR
- SW12: renamed from S12; footprint (none) -> SW_B3F-4000_OMR:SW_B3F-4000_OMR
- SW21: renamed from S21; footprint (none) -> SW_B3F-4000_OMR:SW_B3F-4000_OMR
- SW35: renamed from SWD35; footprint (none) -> SW_B3F-4000_OMR:SW_B3F-4000_OMR
- SW36: renamed from SWX36; footprint (none) -> SW_B3F-4000_OMR:SW_B3F-4000_OMR
- SW46: renamed from SWC46; footprint (none) -> SW_B3F-4000_OMR:SW_B3F-4000_OMR
- renumbered D1 to D00, D15 to D01, D29 to D02, D43 to D03, D57 to D04, D9 to D05, D10 to D06, D11 to D07, D2 to D10, D16 to D11, D30 to D12, D44 to D13, D58 to D14, D12 to D15, D13 to D16, D14 to D17, D3 to D20, D17 to D21, D31 to D22, D45 to D23, D59 to D24, D23 to D25, D24 to D26, D25 to D27, D4 to D30, D18 to D31, D46 to D33, D60 to D34, D26 to D35, D27 to D36, D28 to D37, D5 to D40, D19 to D41, D33 to D42, D47 to D43, D61 to D44, D37 to D45, D38 to D46, D39 to D47, D6 to D50, D20 to D51, D34 to D52, D48 to D53, D62 to D54, D40 to D55, D41 to D56, D42 to D57, D7 to D60, D21 to D61, D35 to D62, D49 to D63, D63 to D64, D51 to D65, D52 to D66, D53 to D67, D8 to D70, D22 to D71, D36 to D72, D50 to D73, D64 to D74, D54 to D75, D55 to D76, D56 to D77, U4 to U1, U5 to U2, U6 to U3, U1 to U6, U2 to U7
Connections:
- net D0: now also U4.3 (D0), U5.18 (O0a)
- net D1: now also U4.4 (D1), U5.16 (O1a)
- net D2: now also U4.7 (D2), U5.14 (O2a)
- net D3: now also U4.8 (D3), U5.12 (O3a)
- net D4: now also U4.13 (D4), U5.9 (O0b)
- net D5: now also U4.14 (D5), U5.7 (O1b)
- net D6: now also U4.17 (D6), U5.5 (O2b)
- net D7: now also U4.18 (D7), U5.3 (O3b)
- net GND: now also C6.1, C7.1, U4.1 (OE), U4.10 (GND), U5.10 (GND)
- net VCC: now also C6.2, C7.2, U4.20 (VCC), U5.20 (VCC)
- net ~{RD}: now also U6.12
- net ~{WR}: now also U6.10
- net ~{GPIO_E}: now reaches U1.12 (O3)
- net ~{GPIO_E}: now also U6.13, U6.9
- net LCD_R/~{W} renamed RD
- new net: J9.5 (Pin_5), U5.11 (I0b)
- new net: J9.6 (Pin_6), U5.13 (I1b)
- new net: J9.7 (Pin_7), U5.15 (I2b)
- new net: J9.8 (Pin_8), U5.17 (I3b)
- new net: J9.1 (Pin_1), U5.2 (I0a)
- new net: J9.2 (Pin_2), U5.4 (I1a)
- new net: J9.3 (Pin_3), U5.6 (I2a)
- new net: J9.4 (Pin_4), U5.8 (I3a)
- new net: J8.1 (Pin_1), U4.2 (O0)
- new net: J8.2 (Pin_2), U4.5 (O1)
- new net: J8.3 (Pin_3), U4.6 (O2)
- new net: J8.4 (Pin_4), U4.9 (O3)
- new net: J8.5 (Pin_5), U4.12 (O4)
- new net: J8.6 (Pin_6), U4.15 (O5)
- new net: J8.7 (Pin_7), U4.16 (O6)
- new net: J8.8 (Pin_8), U4.19 (O7)
- new net: U6.8, U7.9
- new net GPIO_WR: U4.11 (LE), U7.8
- new net ~{GPIO_RD}: U5.1 (OEa), U5.19 (OEb), U6.11
- no-connect marks 29 -> 25
Other:
- note added: "00 01 02 03 04 05 06 07 10 11 12 13 14 15 16 17 Esc 1 2 3 4 5 6 7 8 9 0 - = Bsp CU CD 20 21 22 23 24 25 26 27 30 31 32 33 34 35 36 37 Tab q w e r t y u i o p [ ] Ent CL CR 40 41 42 43 44 45 46 47 50 51 52 53 54 55 56 57 Cap a s d f g h j k l ; ' \ fn ctr alt 60 61 62 63 64 65 66 67 70 71 72 73 74 75 76 77 Sft ` z x c v b n m , . / Sft cmd spc"
- note added: "LCD_R/~{W}"
- note added: "LCD_RS : 0 = status / 1 = data"
- note removed: "0 = status 1 = data"
- note removed: "LCD_RS"
- moved on the sheet: U6B, U7C

Commit message: Update BeanBoard.kicad_sch
Parts:
- J5, J6: footprint Connector_PinSocket_2.54mm:PinSocket_1x07_P2.54mm_Vertical -> Connector_PinSocket_2.54mm:PinSocket_1x03_P2.54mm_Vertical
Changed lines of the file:
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@@
       (effects (font (size 1.27 1.27)) (justify left))
     )
-    (property "Footprint" "Connector_PinSocket_2.54mm:PinSocket_1x07_P2.54mm_Vertical" (at 91.44 157.48 0)
+    (property "Footprint" "Connector_PinSocket_2.54mm:PinSocket_1x03_P2.54mm_Vertical" (at 91.44 157.48 0)
       (effects (font (size 1.27 1.27)) hide)
     )
@@
       (effects (font (size 1.27 1.27)) (justify left))
     )
-    (property "Footprint" "Connector_PinSocket_2.54mm:PinSocket_1x07_P2.54mm_Vertical" (at 91.44 146.05 0)
-      (effects (font (size 1.27 1.27)) hide)
-    )
+    (property "Footprint" "Connector_PinSocket_2.54mm:PinSocket_1x03_P2.54mm_Vertical" (at 91.44 146.05 0)
+      (effects (font (size 1.27 1.27)) hide)
+    )
