File: kicad/BeanBoard.kicad_sch (KiCad schematic)
At the start: 163 parts, among them J1 BZ_Address, J10 Power, J11 Power, J2 BZ_Data, J3 BZ_Control, J4 BZ_Power, J5 BZ_IORQ_enable, J6 BZ_MREQ_enable, J7 LCD, J8 GPO, J9 GPI, SW00 SW_Push_45deg, SW01 SW_Push_45deg, SW02 SW_Push_45deg, SW03 SW_Push_45deg, SW04 SW_Push_45deg, SW05 SW_Push_45deg, SW06 SW_Push_45deg, SW07 SW_Push_45deg, SW10 SW_Push_45deg, SW11 SW_Push_45deg, SW12 SW_Push_45deg, SW13 SW_Push_45deg, SW14 SW_Push_45deg, SW15 SW_Push_45deg, SW16 SW_Push_45deg, SW17 SW_Push_45deg, SW20 SW_Push_45deg, SW21 SW_Push_45deg, SW22 SW_Push_45deg, SW23 SW_Push_45deg, SW24 SW_Push_45deg, SW25 SW_Push_45deg, SW26 SW_Push_45deg, SW27 SW_Push_45deg, SW30 SW_Push_45deg, SW31 SW_Push_45deg, SW32 SW_Push_45deg, SW33 SW_Push_45deg, SW34 SW_Push_45deg, SW35 SW_Push_45deg, SW36 SW_Push_45deg, SW37 SW_Push_45deg, SW40 SW_Push_45deg, SW41 SW_Push_45deg, SW42 SW_Push_45deg, SW43 SW_Push_45deg, SW44 SW_Push_45deg, SW45 SW_Push_45deg, SW46 SW_Push_45deg, SW47 SW_Push_45deg, SW50 SW_Push_45deg, SW51 SW_Push_45deg, SW52 SW_Push_45deg, SW53 SW_Push_45deg, SW54 SW_Push_45deg, SW55 SW_Push_45deg, SW56 SW_Push_45deg, SW57 SW_Push_45deg, SW60 SW_Push_45deg, SW61 SW_Push_45deg, SW62 SW_Push_45deg, SW63 SW_Push_45deg, SW64 SW_Push_45deg, SW65 SW_Push_45deg, SW66 SW_Push_45deg, SW67 SW_Push_45deg, SW70 SW_Push_45deg, SW71 SW_Push_45deg, SW72 SW_Push_45deg, SW73 SW_Push_45deg, SW74 SW_Push_45deg, SW75 SW_Push_45deg, SW76 SW_Push_45deg, SW77 SW_Push_45deg, U1 74LS138, U2 SN74LS373, U3 74LS244, U4 SN74LS373, U5 74LS244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

Commit message: Update BeanBoard.kicad_sch
Parts:
- SW00, SW01, SW02, SW03, SW04, SW05, SW06, SW07, SW10, SW11, SW12, SW13, SW14, SW15, SW16, SW17, SW20, SW21, SW22, SW23, SW24, SW25, SW26, SW27, SW30, SW31, SW32, SW33, SW34, SW35, SW36, SW37, SW40, SW41, SW42, SW43, SW44, SW45, SW46, SW47, SW50, SW51, SW52, SW53, SW54, SW55, SW56, SW57, SW60, SW61, SW62, SW63, SW64, SW65, SW66, SW67, SW70, SW71, SW72, SW73, SW74, SW75, SW76, SW77: footprint SW_B3F-4000_OMR:SW_B3F-4000_OMR -> Button_Switch_Keyboard:SW_Cherry_MX_1.00u_PCB; symbol Switch:SW_Push -> Switch:SW_Push_45deg
Connections:
- net at D37.1 (K), D47.1 (K), D57.1 (K)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: no longer D07.1 (K), D17.1 (K), D27.1 (K)
- net at D77.2 (A): no longer SW77.2
- net at D36.1 (K), D46.1 (K), D56.1 (K)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: no longer D06.1 (K), D16.1 (K), D26.1 (K)
- net at D56.2 (A): no longer SW56.2
- net at SW47.2: no longer D47.2 (A)
- net at D66.2 (A): no longer SW66.2
- net at SW41.2: no longer D41.2 (A)
- net at SW52.2: no longer D52.2 (A)
- net at D34.1 (K), D44.1 (K), D54.1 (K)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: no longer D04.1 (K), D14.1 (K), D24.1 (K)
- net at D64.2 (A): no longer SW64.2
- net at D57.2 (A): no longer SW57.2
- net at D35.1 (K), D45.1 (K), D55.1 (K)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: no longer D05.1 (K), D15.1 (K), D25.1 (K)
- net at D33.1 (K), D43.1 (K), D53.1 (K)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: no longer D03.1 (K), D13.1 (K), D23.1 (K)
- net at D73.2 (A): no longer SW73.2
- net at D14.2 (A): no longer SW14.2
- net at SW62.2: no longer D62.2 (A)
- net at SW17.2: no longer D17.2 (A)
- net at SW22.2: no longer D22.2 (A)
- net at D31.1 (K), D41.1 (K), D51.1 (K)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: no longer D01.1 (K), D11.1 (K), D21.1 (K)
- net at D71.2 (A): no longer SW71.2
- net at D30.1 (K), D40.1 (K), D50.1 (K)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: no longer D00.1 (K), D10.1 (K), D20.1 (K)
- net at D32.1 (K), D42.1 (K), D52.1 (K)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: no longer D02.1 (K), D12.1 (K), D22.1 (K)
- net at SW54.2: no longer D54.2 (A)
- net at SW51.2: no longer D51.2 (A)
- net at SW26.2: no longer D26.2 (A)
- net at SW74.2: no longer D74.2 (A)
- net at SW65.2: no longer D65.2 (A)
- net at D11.2 (A): no longer SW11.2
- net at D63.2 (A): no longer SW63.2
- net at D72.2 (A): no longer SW72.2
- net at D35.2 (A): no longer SW35.2
- net at D30.2 (A): no longer SW30.2
- net at D53.2 (A): no longer SW53.2
- net at D32.2 (A): no longer SW32.2
- net at SW07.2: no longer D07.2 (A)
- net at SW36.2: no longer D36.2 (A)
- net at SW31.2: no longer D31.2 (A)
- net at SW75.2: no longer D75.2 (A)
- net at SW43.2: no longer D43.2 (A)
- net at SW20.2: no longer D20.2 (A)
- net at SW42.2: no longer D42.2 (A)
- net at D60.2 (A): no longer SW60.2
- net at D37.2 (A): no longer SW37.2
- net at SW44.2: no longer D44.2 (A)
- net at SW45.2: no longer D45.2 (A)
- net at D12.2 (A): no longer SW12.2
- net at SW10.2: no longer D10.2 (A)
- net at SW05.2: no longer D05.2 (A)
- net at SW46.2: no longer D46.2 (A)
- net at SW50.2: no longer D50.2 (A)
- net at D16.2 (A): no longer SW16.2
- net at D24.2 (A): no longer SW24.2
- net at SW06.2: no longer D06.2 (A)
- net at SW67.2: no longer D67.2 (A)
- net at SW21.2: no longer D21.2 (A)
- net at SW13.2: no longer D13.2 (A)
- net at D76.2 (A): no longer SW76.2
- net at D70.2 (A): no longer SW70.2
- net at D15.2 (A): no longer SW15.2
- net at D23.2 (A): no longer SW23.2
- net at D40.2 (A): no longer SW40.2
- net at D33.2 (A): no longer SW33.2
- net at SW25.2: no longer D25.2 (A)
- net at D55.2 (A): no longer SW55.2
- net at SW27.2: no longer D27.2 (A)
- net at SW34.2: no longer D34.2 (A)
- net at D61.2 (A): no longer SW61.2
- now unconnected: SW00.1, SW01.1, SW02.1, SW03.1, SW04.1, SW05.1, SW06.1, SW07.1, SW10.1, SW11.1, SW12.1, SW13.1, SW14.1, SW15.1, SW16.1, SW17.1, SW20.1, SW21.1, SW22.1, SW23.1, SW24.1, SW25.1, SW26.1, SW27.1, SW30.1, SW31.1, SW32.1, SW33.1, SW34.1, SW35.1, SW36.1, SW37.1, SW40.1, SW41.1, SW42.1, SW43.1, SW44.1, SW45.1, SW46.1, SW47.1, SW50.1, SW51.1, SW52.1, SW53.1, SW54.1, SW55.1, SW56.1, SW57.1, SW60.1, SW61.1, SW62.1, SW63.1, SW64.1, SW65.1, SW66.1, SW67.1, SW70.1, SW71.1, SW72.1, SW73.1, SW74.1, SW75.1, SW76.1, SW77.1, U2.12 (O4), U2.15 (O5), U2.16 (O6), U2.19 (O7), U2.2 (O0), U2.5 (O1), U2.6 (O2), U2.9 (O3)
Other:
- moved on the sheet: D00, D01, D02, D03, D04, D05, D06, D07, D10, D11, D12, D13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

Commit message: Update BeanBoard.kicad_sch
Connections:
- net at D14.2 (A): now also SW14.2
- net at SW17.2: now also D17.2 (A)
- net at SW22.2: now also D22.2 (A)
- net at SW26.2: now also D26.2 (A)
- net at D11.2 (A): now also SW11.2
- net at SW07.2: now also D07.2 (A)
- net at SW20.2: now also D20.2 (A)
- net at D12.2 (A): now also SW12.2
- net at SW10.2: now also D10.2 (A)
- net at SW05.2: now also D05.2 (A)
- net at D16.2 (A): now also SW16.2
- net at D24.2 (A): now also SW24.2
- net at SW06.2: now also D06.2 (A)
- net at SW21.2: now also D21.2 (A)
- net at SW13.2: now also D13.2 (A)
- net at D15.2 (A): now also SW15.2
- net at D23.2 (A): now also SW23.2
- net at SW25.2: now also D25.2 (A)
- net at SW27.2: now also D27.2 (A)
Other:
- moved on the sheet: D00, D01, D02, D03, D04, D05, D06, D07, D10, D11, D12, D13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

Commit message: Update BeanBoard.kicad_sch
Connections:
- net at D77.2 (A): now also SW77.2
- net at D56.2 (A): now also SW56.2
- net at SW47.2: now also D47.2 (A)
- net at D66.2 (A): now also SW66.2
- net at SW41.2: now also D41.2 (A)
- net at SW52.2: now also D52.2 (A)
- net at D64.2 (A): now also SW64.2
- net at D57.2 (A): now also SW57.2
- net at D73.2 (A): now also SW73.2
- net at SW62.2: now also D62.2 (A)
- net at D71.2 (A): now also SW71.2
- net at SW54.2: now also D54.2 (A)
- net at SW51.2: now also D51.2 (A)
- net at SW74.2: now also D74.2 (A)
- net at SW65.2: now also D65.2 (A)
- net at D63.2 (A): now also SW63.2
- net at D72.2 (A): now also SW72.2
- net at D35.2 (A): now also SW35.2
- net at D30.2 (A): now also SW30.2
- net at D53.2 (A): now also SW53.2
- net at D32.2 (A): now also SW32.2
- net at SW36.2: now also D36.2 (A)
- net at SW31.2: now also D31.2 (A)
- net at SW75.2: now also D75.2 (A)
- net at SW43.2: now also D43.2 (A)
- net at SW42.2: now also D42.2 (A)
- net at D60.2 (A): now also SW60.2
- net at D37.2 (A): now also SW37.2
- net at SW44.2: now also D44.2 (A)
- net at SW45.2: now also D45.2 (A)
- net at SW46.2: now also D46.2 (A)
- net at SW50.2: now also D50.2 (A)
- net at SW67.2: now also D67.2 (A)
- net at D76.2 (A): now also SW76.2
- net at D70.2 (A): now also SW70.2
- net at D40.2 (A): now also SW40.2
- net at D33.2 (A): now also SW33.2
- net at D55.2 (A): now also SW55.2
- net at SW34.2: now also D34.2 (A)
- net at D61.2 (A): now also SW61.2
- new net: R6.2, U3.13 (I1b)
- new net: R8.2, U3.17 (I3b)
- new net: R5.2, U3.11 (I0b)
- new net: R7.2, U3.15 (I2b)
- new net: R1.2, U3.2 (I0a)
- new net: R2.2, U3.4 (I1a)
- new net: R3.2, U3.6 (I2a)
- new net: R4.2, U3.8 (I3a)
- now unconnected: D30.1 (K), D31.1 (K), D32.1 (K), D33.1 (K), D34.1 (K), D35.1 (K), D36.1 (K), D37.1 (K), D40.1 (K), D41.1 (K), D42.1 (K), D43.1 (K), D44.1 (K), D45.1 (K), D46.1 (K), D47.1 (K), D50.1 (K), D51.1 (K), D52.1 (K), D53.1 (K), D54.1 (K), D55.1 (K), D56.1 (K), D57.1 (K), D60.1 (K), D61.1 (K), D62.1 (K), D63.1 (K), D64.1 (K), D65.1 (K), D66.1 (K), D67.1 (K), D70.1 (K), D71.1 (K), D72.1 (K), D73.1 (K), D74.1 (K), D75.1 (K), D76.1 (K), D77.1 (K)
Other:
- moved on the sheet: D00, D01, D02, D03, D04, D05, D06, D07, D10, D11, D12, D13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

Commit message: Update BeanBoard.kicad_sch
Connections:
- net at SW04.1: now also SW00.1, SW01.1, SW02.1, SW03.1, SW05.1, SW06.1, SW07.1, U2.2 (O0)
- net at D77.1 (K): now also D07.1 (K), D17.1 (K), D27.1 (K), D37.1 (K), D47.1 (K), D57.1 (K), D67.1 (K), R8.2, U3.17 (I3b)
- net at D56.1 (K): now also D06.1 (K), D16.1 (K), D26.1 (K), D36.1 (K), D46.1 (K), D66.1 (K), D76.1 (K), R7.2, U3.15 (I2b)
- net at SW47.1: now also SW40.1, SW41.1, SW42.1, SW43.1, SW44.1, SW45.1, SW46.1, U2.12 (O4)
- net at SW56.1: now also SW50.1, SW51.1, SW52.1, SW53.1, SW54.1, SW55.1, SW57.1, U2.15 (O5)
- net at D64.1 (K): now also D04.1 (K), D14.1 (K), D24.1 (K), D34.1 (K), D44.1 (K), D54.1 (K), D74.1 (K), R5.2, U3.11 (I0b)
- net at SW77.1: now also SW70.1, SW71.1, SW72.1, SW73.1, SW74.1, SW75.1, SW76.1, U2.19 (O7)
- net at R6.2, U3.13 (I1b): now also D05.1 (K), D15.1 (K), D25.1 (K), D35.1 (K), D45.1 (K), D55.1 (K), D65.1 (K), D75.1 (K)
- net at D73.1 (K): now also D03.1 (K), D13.1 (K), D23.1 (K), D33.1 (K), D43.1 (K), D53.1 (K), D63.1 (K), R4.2, U3.8 (I3a)
- net at SW66.1: now also SW60.1, SW61.1, SW62.1, SW63.1, SW64.1, SW65.1, SW67.1, U2.16 (O6)
- net at SW17.1: now also SW10.1, SW11.1, SW12.1, SW13.1, SW14.1, SW15.1, SW16.1, U2.5 (O1)
- net at SW22.1: now also SW20.1, SW21.1, SW23.1, SW24.1, SW25.1, SW26.1, SW27.1, U2.6 (O2)
- net at D71.1 (K): now also D01.1 (K), D11.1 (K), D21.1 (K), D31.1 (K), D41.1 (K), D51.1 (K), D61.1 (K), R2.2, U3.4 (I1a)
- net at R1.2, U3.2 (I0a): now also D00.1 (K), D10.1 (K), D20.1 (K), D30.1 (K), D40.1 (K), D50.1 (K), D60.1 (K), D70.1 (K)
- net at R3.2, U3.6 (I2a): now also D02.1 (K), D12.1 (K), D22.1 (K), D32.1 (K), D42.1 (K), D52.1 (K), D62.1 (K), D72.1 (K)
- net at SW30.1: now also SW31.1, SW32.1, SW33.1, SW34.1, SW35.1, SW36.1, SW37.1, U2.9 (O3)
Other:
- moved on the sheet: C2, C3, D35, D36, D37, D50, D51, D52, D53, D54, D55, D56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
