File: kicad/BeanBoard.kicad_sch (KiCad schematic)
At the start: 163 parts, among them J1 BZ_Address, J10 Power, J11 Power, J2 BZ_Data, J3 BZ_Control, J4 BZ_Power, J5 BZ_IORQ_enable, J6 BZ_MREQ_enable, J7 LCD, J8 GPO, J9 GPI, SW00 SW_Push_45deg, SW01 SW_Push_45deg, SW02 SW_Push_45deg, SW03 SW_Push_45deg, SW04 SW_Push_45deg, SW05 SW_Push_45deg, SW06 SW_Push_45deg, SW07 SW_Push_45deg, SW10 SW_Push_45deg, SW11 SW_Push_45deg, SW12 SW_Push_45deg, SW13 SW_Push_45deg, SW14 SW_Push_45deg, SW15 SW_Push_45deg, SW16 SW_Push_45deg, SW17 SW_Push_45deg, SW20 SW_Push_45deg, SW21 SW_Push_45deg, SW22 SW_Push_45deg, SW23 SW_Push_45deg, SW24 SW_Push_45deg, SW25 SW_Push_45deg, SW26 SW_Push_45deg, SW27 SW_Push_45deg, SW30 SW_Push_45deg, SW31 SW_Push_45deg, SW32 SW_Push_45deg, SW33 SW_Push_45deg, SW34 SW_Push_45deg, SW35 SW_Push_45deg, SW36 SW_Push_45deg, SW37 SW_Push_45deg, SW40 SW_Push_45deg, SW41 SW_Push_45deg, SW42 SW_Push_45deg, SW43 SW_Push_45deg, SW44 SW_Push_45deg, SW45 SW_Push_45deg, SW46 SW_Push_45deg, SW47 SW_Push_45deg, SW50 SW_Push_45deg, SW51 SW_Push_45deg, SW52 SW_Push_45deg, SW53 SW_Push_45deg, SW54 SW_Push_45deg, SW55 SW_Push_45deg, SW56 SW_Push_45deg, SW57 SW_Push_45deg, SW60 SW_Push_45deg, SW61 SW_Push_45deg, SW62 SW_Push_45deg, SW63 SW_Push_45deg, SW64 SW_Push_45deg, SW65 SW_Push_45deg, SW66 SW_Push_45deg, SW67 SW_Push_45deg, SW70 SW_Push_45deg, SW71 SW_Push_45deg, SW72 SW_Push_45deg, SW73 SW_Push_45deg, SW74 SW_Push_45deg, SW75 SW_Push_45deg, SW76 SW_Push_45deg, SW77 SW_Push_45deg, U1 74LS138, U2 SN74LS373, U3 74LS244, U4 SN74LS373, U5 74LS244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

Commit message: Update BeanBoard.kicad_sch
Other:
- note removed: "00 01 02 03 04 05 06 07 10 11 12 13 14 15 Esc 1 2 3 4 5 6 7 8 9 0 - = Bsp"
- note removed: "16 CU"
- note removed: "17 CD"
- note removed: "20 21 22 23 24 25 26 27 30 31 32 33 34 35 Tab q w e r t y u i o p [ ] Ent"
- note removed: "36 CL"
- note removed: "37 CR"
- note removed: "40 41 42 43 44 45 46 47 50 51 52 53 54 Cap a s d f g h j k l ; ' \"
- note removed: "55 56 57 75 76 77 fn ctr alt cmd spc"
- note removed: "60 61 62 63 64 65 66 67 70 71 72 73 74 Sft ` z x c v b n m , . / Sft"
- moved on the sheet: C1, C2, C3, C6, C7, D00, D01, D02, D03, D04, D05, D06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

Commit message: Update BeanBoard.kicad_sch
Parts:
- removed J11: Power, Connector_PinSocket_2.54mm:PinSocket_1x02_P2.54mm_Vertical, symbol Connector:Conn_01x02_Socket
- added J11: Barrel_Jack_Switch, Connector_BarrelJack:BarrelJack_CUI_PJ-102AH_Horizontal, symbol Connector:Barrel_Jack_Switch
- added J12: GPIO_RW, Connector_PinSocket_2.54mm:PinSocket_1x02_P2.54mm_Vertical, symbol Connector:Conn_01x02_Socket
Connections:
- net ~{GPIO_RD}: now also J12.1 (Pin_1)
- net ~{GPIO_WR}: now reaches U6.8, U7.9
- net ~{GPIO_WR}: now also J12.2 (Pin_2)
Other:
- note removed: "~{M1} should enable / disable IO on E3 - but we haven't made that available on BeanZee"
- moved on the sheet: J10
Changed lines of the file:
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@@
   (junction (at 330.2 118.11) (diameter 0) (color 0 0 0 0)
   )
+  (junction (at 125.73 118.11) (diameter 0) (color 0 0 0 0)
+  )
   (junction (at 314.96 147.32) (diameter 0) (color 0 0 0 0)
   )
@@
     (stroke (width 0) (type default))
   )
+  (wire (pts (xy 125.73 118.11) (xy 121.92 118.11))
+    (stroke (width 0) (type default))
+  )
   (wire (pts (xy 299.72 118.11) (xy 299.72 132.08))
     (stroke (width 0) (type default))
@@
     (stroke (width 0) (type default))
   )
-  (wire (pts (xy 83.82 204.47) (xy 83.82 207.01))
+  (wire (pts (xy 205.74 219.71) (xy 205.74 222.25))
     (stroke (width 0) (type default))
   )
@@
     (stroke (width 0) (type default))
   )
-  (wire (pts (xy 50.8 201.93) (xy 66.04 201.93))
-    (stroke (width 0) (type default))
-  )
   (wire (pts (xy 173.99 241.3) (xy 180.34 241.3))
     (stroke (width 0) (type default))
@@
     (stroke (width 0) (type default))
   )
+  (wire (pts (xy 208.28 271.78) (xy 220.98 271.78))
+    (stroke (width 0) (type default))
+  )
   (wire (pts (xy 378.46 107.95) (xy 378.46 113.03))
     (stroke (width 0) (type default))
@@
     (stroke (width 0) (type default))
   )
-  (wire (pts (xy 130.81 118.11) (xy 121.92 118.11))
+  (wire (pts (xy 130.81 118.11) (xy 125.73 118.11))
     (stroke (width 0) (type default))
   )
@@
     (stroke (width 0) (type default))
   )
-  (wire (pts (xy 50.8 204.47) (xy 66.04 204.47))
-    (stroke (width 0) (type default))
-  )
   (wire (pts (xy 330.2 177.8) (xy 330.2 182.88))
     (stroke (width 0) (type default))
@@
     (stroke (width 0) (type default))
   )
-  (wire (pts (xy 83.82 199.39) (xy 83.82 201.93))
+  (wire (pts (xy 205.74 214.63) (xy 205.74 217.17))
     (stroke (width 0) (type default))
   )
@@
     (stroke (width 0) (type default))
   )
-  (wire (pts (xy 83.82 201.93) (xy 99.06 201.93))
+  (wire (pts (xy 205.74 217.17) (xy 220.98 217.17))
     (stroke (width 0) (type default))
   )
@@
     (stroke (width 0) (type default))
   )
+  (wire (pts (xy 208.28 274.32) (xy 220.98 274.32))
+    (stroke (width 0) (type default))
+  )
   (wire (pts (xy 205.74 251.46) (xy 210.82 251.46))
     (stroke (width 0) (type default))
@@
     (stroke (width 0) (type default))
   )
-  (wire (pts (xy 83.82 204.47) (xy 99.06 204.47))
+  (wire (pts (xy 205.74 219.71) (xy 220.98 219.71))
     (stroke (width 0) (type default))
   )
@@
     (stroke (width 0) (type default))
   )
+  (wire (pts (xy 125.73 129.54) (xy 125.73 118.11))
+    (stroke (width 0) (type default))
+  )
   (wire (pts (xy 128.27 180.34) (xy 146.05 180.34))
     (stroke (width 0) (type default))
@@
     (stroke (width 0) (type default))
   )
+  (wire (pts (xy 154.94 129.54) (xy 125.73 129.54))
+    (stroke (width 0) (type default))
+  )
   (wire (pts (xy 224.79 119.38) (xy 231.14 119.38))
     (stroke (width 0) (type default))
@@
     (stroke (width 0) (type default))
   )
-  (text "Row 0" (at 397.51 72.39 0)
-    (effects (font (size 1.27 1.27)) (justify left bottom))
+  (rectangle (start 24.13 137.16) (end 118.11 186.69)
+    (stroke (width 0) (type dot))
+    (fill (type none))
   )
-  (text "~{M1} should enable / disable IO on E3\n- but we haven't made that available on BeanZee"
-    (at 22.86 24.13 0)
+  (text "Row 0" (at 397.51 72.39 0)
     (effects (font (size 1.27 1.27)) (justify left bottom))
   )
@@
     (effects (font (size 1.27 1.27)) (justify right bottom))
   )
+  (label "~{GPIO_RD}" (at 208.28 271.78 0) (fields_autoplaced)
+    (effects (font (size 1.27 1.27)) (justify left bottom))
+  )
   (label "~{WR}" (at 59.69 168.91 180) (fields_autoplaced)
     (effects (font (size 1.27 1.27)) (justify right bottom))
@@
     (effects (font (size 1.27 1.27)) (justify left bottom))
   )
+  (label "~{GPIO_WR}" (at 208.28 274.32 0) (fields_autoplaced)
+    (effects (font (size 1.27 1.27)) (justify left bottom))
+  )
   (label "~{RD}" (at 38.1 96.52 0) (fields_autoplaced)
     (effects (font (size 1.27 1.27)) (justify left bottom))
@@
     (effects (font (size 1.27 1.27)) (justify right bottom))
   )
+  (label "~{GPIO_WR}" (at 154.94 129.54 180) (fields_autoplaced)
+    (effects (font (size 1.27 1.27)) (justify right bottom))
+  )
   (label "LCD_E" (at 130.81 157.48 0) (fields_autoplaced)
     (effects (font (size 1.27 1.27)) (justify left bottom))
@@
     )
   )
+  (symbol (lib_id "Connector:Conn_01x02_Socket") (at 226.06 271.78 0) (unit 1)
+    (in_bom yes) (on_board yes) (dnp no) (fields_autoplaced)
+    (property "Reference" "J12" (at 227.33 271.78 0)
+      (effects (font (size 1.27 1.27)) (justify left))
+    )
+    (property "Value" "GPIO_RW" (at 227.33 274.32 0)
+      (effects (font (size 1.27 1.27)) (justify left))
+    )
+    (property "Footprint" "Connector_PinSocket_2.54mm:PinSocket_1x02_P2.54mm_Vertical" (at 226.06 271.78 0)
+      (effects (font (size 1.27 1.27)) hide)
+    )
+    (property "Datasheet" "~" (at 226.06 271.78 0)
+      (effects (font (size 1.27 1.27)) hide)
+    )
+    (pin "2")
+    (pin "1")
+    (instances
+      (project "BeanBoard"
+        (path "/3defbfd6-25f4-40d7-986c-89ce878d27b9"
+          (reference "J12") (unit 1)
+        )
+      )
+    )
+  )
   (symbol (lib_id "Device:C") (at 25.4 241.3 90) (unit 1)
     (in_bom yes) (on_board yes) (dnp no) (fields_autoplaced)
@@
     )
   )
+  (symbol (lib_id "Connector:Barrel_Jack_Switch") (at 33.02 204.47 0) (unit 1)
+    (in_bom yes) (on_board yes) (dnp no) (fields_autoplaced)
+    (property "Reference" "J11" (at 33.02 195.58 0)
+      (effects (font (size 1.27 1.27)))
+    )
+    (property "Value" "Barrel_Jack_Switch" (at 33.02 198.12 0)
+      (effects (font (size 1.27 1.27)))
+    )
+    (property "Footprint" "Connector_BarrelJack:BarrelJack_CUI_PJ-102AH_Horizontal" (at 34.29 205.486 0)
+      (effects (font (size 1.27 1.27)) hide)
+    )
+    (property "Datasheet" "~" (at 34.29 205.486 0)
+      (effects (font (size 1.27 1.27)) hide)
+    )
+    (pin "3")
+    (pin "1")
+    (pin "2")
+    (instances
+      (project "BeanBoard"
+        (path "/3defbfd6-25f4-40d7-986c-89ce878d27b9"
+          (reference "J11") (unit 1)
+        )
+      )
+    )
+  )
   (symbol (lib_id "Diode:1N4148") (at 311.15 90.17 180) (unit 1)
     (in_bom yes) (on_board yes) (dnp no) (fields_autoplaced)
@@
     )
   )
-  (symbol (lib_name "GND_2") (lib_id "power:GND") (at 83.82 207.01 0) (unit 1)
+  (symbol (lib_name "GND_2") (lib_id "power:GND") (at 205.74 222.25 0) (unit 1)
     (in_bom yes) (on_board yes) (dnp no)
-    (property "Reference" "#PWR030" (at 83.82 213.36 0)
+    (property "Reference" "#PWR030" (at 205.74 228.6 0)
       (effects (font (size 1.27 1.27)) hide)
     )
-    (property "Value" "GND" (at 83.82 210.82 0)
+    (property "Value" "GND" (at 205.74 226.06 0)
       (effects (font (size 1.27 1.27)))
     )
-    (property "Footprint" "" (at 83.82 207.01 0)
+    (property "Footprint" "" (at 205.74 222.25 0)
       (effects (font (size 1.27 1.27)) hide)
     )
-    (property "Datasheet" "" (at 83.82 207.01 0)
+    (property "Datasheet" "" (at 205.74 222.25 0)
       (effects (font (size 1.27 1.27)) hide)
     )
@@
     )
   )
-  (symbol (lib_id "power:VCC") (at 83.82 199.39 0) (unit 1)
+  (symbol (lib_id "power:VCC") (at 205.74 214.63 0) (unit 1)
     (in_bom yes) (on_board yes) (dnp no)
-    (property "Reference" "#PWR029" (at 83.82 203.2 0)
+    (property "Reference" "#PWR029" (at 205.74 218.44 0)
       (effects (font (size 1.27 1.27)) hide)
     )
-    (property "Value" "VCC" (at 83.82 195.58 0)
+    (property "Value" "VCC" (at 205.74 210.82 0)
       (effects (font (size 1.27 1.27)))
     )
-    (property "Footprint" "" (at 83.82 199.39 0)
+    (property "Footprint" "" (at 205.74 214.63 0)
       (effects (font (size 1.27 1.27)) hide)
     )
-    (property "Datasheet" "" (at 83.82 199.39 0)
+    (property "Datasheet" "" (at 205.74 214.63 0)
       (effects (font (size 1.27 1.27)) hide)
     )
@@
     )
   )
-  (symbol (lib_id "Connector:Conn_01x02_Socket") (at 71.12 201.93 0) (unit 1)
-    (in_bom yes) (on_board yes) (dnp no) (fields_autoplaced)
-    (property "Reference" "J11" (at 72.39 201.93 0)
-      (effects (font (size 1.27 1.27)) (justify left))
-    )
-    (property "Value" "Power" (at 72.39 204.47 0)
-      (effects (font (size 1.27 1.27)) (justify left))
-    )
-    (property "Footprint" "Connector_PinSocket_2.54mm:PinSocket_1x02_P2.54mm_Vertical" (at 71.12 201.93 0)
-      (effects (font (size 1.27 1.27)) hide)
-    )
-    (property "Datasheet" "~" (at 71.12 201.93 0)
-      (effects (font (size 1.27 1.27)) hide)
-    )
-    (pin "2")
-    (pin "1")
-    (instances
-      (project "BeanBoard"
-        (path "/3defbfd6-25f4-40d7-986c-89ce878d27b9"
-          (reference "J11") (unit 1)
-        )
-      )
-    )
-  )
   (symbol (lib_id "power:GND") (at 138.43 139.7 0) (unit 1)
     (in_bom yes) (on_board yes) (dnp no)
@@
     )
   )
-  (symbol (lib_id "Connector:Conn_01x02_Socket") (at 104.14 201.93 0) (unit 1)
+  (symbol (lib_id "Connector:Conn_01x02_Socket") (at 226.06 217.17 0) (unit 1)
     (in_bom yes) (on_board yes) (dnp no) (fields_autoplaced)
-    (property "Reference" "J10" (at 105.41 201.93 0)
+    (property "Reference" "J10" (at 227.33 217.17 0)
       (effects (font (size 1.27 1.27)) (justify left))
     )
-    (property "Value" "Power" (at 105.41 204.47 0)
+    (property "Value" "Power" (at 227.33 219.71 0)
       (effects (font (size 1.27 1.27)) (justify left))
     )
-    (property "Footprint" "Connector_PinSocket_2.54mm:PinSocket_1x02_P2.54mm_Vertical" (at 104.14 201.93 0)
+    (property "Footprint" "Connector_PinSocket_2.54mm:PinSocket_1x02_P2.54mm_Vertical" (at 226.06 217.17 0)
       (effects (font (size 1.27 1.27)) hide)
     )
-    (property "Datasheet" "~" (at 104.14 201.93 0)
+    (property "Datasheet" "~" (at 226.06 217.17 0)
       (effects (font (size 1.27 1.27)) hide)
     )

Commit message: Update BeanBoard.kicad_sch
Parts:
- removed J10: Power, Connector_PinSocket_2.54mm:PinSocket_1x02_P2.54mm_Vertical, symbol Connector:Conn_01x02_Socket
- removed J12: GPIO_RW, Connector_PinSocket_2.54mm:PinSocket_1x02_P2.54mm_Vertical, symbol Connector:Conn_01x02_Socket
- removed J8: GPO, Connector_PinSocket_2.54mm:PinSocket_1x08_P2.54mm_Vertical, symbol Connector:Conn_01x08_Socket
- removed J9: GPI, Connector_PinSocket_2.54mm:PinSocket_1x08_P2.54mm_Vertical, symbol Connector:Conn_01x08_Socket
- added J13: Conn_02x10_Row_Letter_First, symbol Connector_Generic:Conn_02x10_Row_Letter_First
Connections:
- net GND: now also J11.2, J13.b10 (Pin_b10)
- net VCC: now also J11.1, J13.a10 (Pin_a10)
- net ~{GPIO_RD}: now also J13.b9 (Pin_b9)
- net ~{GPIO_WR}: now also J13.a9 (Pin_a9)
- net at U5.11 (I0b): now also J13.b5 (Pin_b5)
- net at U5.13 (I1b): now also J13.b6 (Pin_b6)
- net at U5.15 (I2b): now also J13.b7 (Pin_b7)
- net at U5.17 (I3b): now also J13.b8 (Pin_b8)
- net at U5.2 (I0a): now also J13.b1 (Pin_b1)
- net at U5.4 (I1a): now also J13.b2 (Pin_b2)
- net at U5.6 (I2a): now also J13.b3 (Pin_b3)
- net at U5.8 (I3a): now also J13.b4 (Pin_b4)
- net at U4.2 (O0): now also J13.a1 (Pin_a1)
- net at U4.5 (O1): now also J13.a2 (Pin_a2)
- net at U4.6 (O2): now also J13.a3 (Pin_a3)
- net at U4.9 (O3): now also J13.a4 (Pin_a4)
- net at U4.12 (O4): now also J13.a5 (Pin_a5)
- net at U4.15 (O5): now also J13.a6 (Pin_a6)
- net at U4.16 (O6): now also J13.a7 (Pin_a7)
- net at U4.19 (O7): now also J13.a8 (Pin_a8)
- no-connect marks 25 -> 26

Commit message: Update BeanBoard.kicad_sch
Parts:
- J13: footprint (none) -> Connector_PinSocket_2.54mm:PinSocket_2x10_P2.54mm_Vertical
Changed lines of the file:
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@@
       (effects (font (size 1.27 1.27)) hide)
     )
-    (property "Footprint" "" (at 220.98 246.38 0)
+    (property "Footprint" "Connector_PinSocket_2.54mm:PinSocket_2x10_P2.54mm_Vertical" (at 220.98 246.38 0)
       (effects (font (size 1.27 1.27)) hide)
     )

Commit message: Update BeanBoard.kicad_sch
Parts:
- removed J13: Conn_02x10_Row_Letter_First, Connector_PinSocket_2.54mm:PinSocket_2x10_P2.54mm_Vertical, symbol Connector_Generic:Conn_02x10_Row_Letter_First
- added C8: 100uF, Capacitor_THT:CP_Radial_D5.0mm_P2.00mm, symbol Device:C_Polarized
- added J8, J9: Conn_01x10_Socket, Connector_PinSocket_2.54mm:PinSocket_1x10_P2.54mm_Vertical, symbol Connector:Conn_01x10_Socket
Connections:
- net GND: now also C8.2, J9.10 (Pin_10)
- net VCC: now also C8.1, J8.10 (Pin_10)
- net ~{GPIO_RD}: now also J9.9 (Pin_9)
- net ~{GPIO_WR}: now also J8.9 (Pin_9)
- net at U5.11 (I0b): now also J9.5 (Pin_5)
- net at U5.13 (I1b): now also J9.6 (Pin_6)
- net at U5.15 (I2b): now also J9.7 (Pin_7)
- net at U5.17 (I3b): now also J9.8 (Pin_8)
- net at U5.2 (I0a): now also J9.1 (Pin_1)
- net at U5.4 (I1a): now also J9.2 (Pin_2)
- net at U5.6 (I2a): now also J9.3 (Pin_3)
- net at U5.8 (I3a): now also J9.4 (Pin_4)
- net at U4.2 (O0): now also J8.1 (Pin_1)
- net at U4.5 (O1): now also J8.2 (Pin_2)
- net at U4.6 (O2): now also J8.3 (Pin_3)
- net at U4.9 (O3): now also J8.4 (Pin_4)
- net at U4.12 (O4): now also J8.5 (Pin_5)
- net at U4.15 (O5): now also J8.6 (Pin_6)
- net at U4.16 (O6): now also J8.7 (Pin_7)
- net at U4.19 (O7): now also J8.8 (Pin_8)
Changed lines of the file:
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@@
   (junction (at 375.92 191.77) (diameter 0) (color 0 0 0 0)
   )
+  (junction (at 50.8 201.93) (diameter 0) (color 0 0 0 0)
+  )
   (junction (at 314.96 132.08) (diameter 0) (color 0 0 0 0)
   )
@@
   (junction (at 332.74 107.95) (diameter 0) (color 0 0 0 0)
   )
+  (junction (at 50.8 209.55) (diameter 0) (color 0 0 0 0)
+  )
   (junction (at 345.44 147.32) (diameter 0) (color 0 0 0 0)
   )
@@
     (stroke (width 0) (type default))
   )
+  (wire (pts (xy 50.8 212.09) (xy 50.8 209.55))
+    (stroke (width 0) (type default))
+  )
   (wire (pts (xy 21.59 274.32) (xy 69.85 274.32))
     (stroke (width 0) (type default))
@@
     (stroke (width 0) (type default))
   )
+  (wire (pts (xy 50.8 209.55) (xy 58.42 209.55))
+    (stroke (width 0) (type default))
+  )
   (wire (pts (xy 58.42 35.56) (xy 58.42 38.1))
     (stroke (width 0) (type default))
@@
     (stroke (width 0) (type default))
   )
+  (wire (pts (xy 50.8 201.93) (xy 58.42 201.93))
+    (stroke (width 0) (type default))
+  )
   (wire (pts (xy 260.35 224.79) (xy 260.35 228.6))
     (stroke (width 0) (type default))
@@
     )
   )
+  (symbol (lib_id "Device:C_Polarized") (at 58.42 205.74 0) (unit 1)
+    (in_bom yes) (on_board yes) (dnp no) (fields_autoplaced)
+    (property "Reference" "C8" (at 62.23 204.851 0)
+      (effects (font (size 1.27 1.27)) (justify left) hide)
+    )
+    (property "Value" "100uF" (at 62.23 206.121 0)
+      (effects (font (size 1.27 1.27)) (justify left))
+    )
+    (property "Footprint" "Capacitor_THT:CP_Radial_D5.0mm_P2.00mm" (at 59.3852 209.55 0)
+      (effects (font (size 1.27 1.27)) hide)
+    )
+    (property "Datasheet" "~" (at 58.42 205.74 0)
+      (effects (font (size 1.27 1.27)) hide)
+    )
+    (pin "1")
+    (pin "2")
+    (instances
+      (project "BeanBoard"
+        (path "/3defbfd6-25f4-40d7-986c-89ce878d27b9"
+          (reference "C8") (unit 1)
+        )
+      )
+    )
+  )
   (symbol (lib_id "Switch:SW_Push_45deg") (at 289.56 129.54 0) (unit 1)
     (in_bom yes) (on_board yes) (dnp no) (fields_autoplaced)
@@
     )
   )
-  (symbol (lib_id "power:VCC") (at 50.8 199.39 0) (unit 1)
+  (symbol (lib_id "Connector:Conn_01x10_Socket") (at 223.52 246.38 0) (mirror y) (unit 1)
     (in_bom yes) (on_board yes) (dnp no)
-    (property "Reference" "#PWR031" (at 50.8 203.2 0)
-      (effects (font (size 1.27 1.27)) hide)
+    (property "Reference" "J9" (at 227.33 231.14 0)
+      (effects (font (size 1.27 1.27)) (justify left))
     )
-    (property "Value" "VCC" (at 50.8 195.58 0)
-      (effects (font (size 1.27 1.27)))
+    (property "Value" "Conn_01x10_Socket" (at 243.84 228.6 0)
+      (effects (font (size 1.27 1.27)) (justify left) hide)
     )
-    (property "Footprint" "" (at 50.8 199.39 0)
+    (property "Footprint" "Connector_PinSocket_2.54mm:PinSocket_1x10_P2.54mm_Vertical" (at 223.52 246.38 0)
       (effects (font (size 1.27 1.27)) hide)
     )
-    (property "Datasheet" "" (at 50.8 199.39 0)
+    (property "Datasheet" "~" (at 223.52 246.38 0)
       (effects (font (size 1.27 1.27)) hide)
     )
+    (pin "9")
     (pin "1")
+    (pin "8")
+    (pin "4")
+    (pin "2")
+    (pin "3")
+    (pin "10")
+    (pin "6")
+    (pin "7")
+    (pin "5")
     (instances
       (project "BeanBoard"
         (path "/3defbfd6-25f4-40d7-986c-89ce878d27b9"
-          (reference "#PWR031") (unit 1)
+          (reference "J9") (unit 1)
         )
       )
     )
   )
-  (symbol (lib_id "Connector_Generic:Conn_02x10_Row_Letter_First") (at 220.98 246.38 0) (unit 1)
-    (in_bom yes) (on_board yes) (dnp no) (fields_autoplaced)
-    (property "Reference" "J13" (at 222.25 229.87 0)
-      (effects (font (size 1.27 1.27)))
-    )
-    (property "Value" "Conn_02x10_Row_Letter_First" (at 222.25 232.41 0)
+  (symbol (lib_id "power:VCC") (at 50.8 199.39 0) (unit 1)
+    (in_bom yes) (on_board yes) (dnp no)
+    (property "Reference" "#PWR031" (at 50.8 203.2 0)
       (effects (font (size 1.27 1.27)) hide)
     )
-    (property "Footprint" "Connector_PinSocket_2.54mm:PinSocket_2x10_P2.54mm_Vertical" (at 220.98 246.38 0)
+    (property "Value" "VCC" (at 50.8 195.58 0)
+      (effects (font (size 1.27 1.27)))
+    )
+    (property "Footprint" "" (at 50.8 199.39 0)
       (effects (font (size 1.27 1.27)) hide)
     )
-    (property "Datasheet" "~" (at 220.98 246.38 0)
+    (property "Datasheet" "" (at 50.8 199.39 0)
       (effects (font (size 1.27 1.27)) hide)
     )
-    (pin "a2")
-    (pin "a3")
-    (pin "a9")
-    (pin "a8")
-    (pin "a5")
-    (pin "a4")
-    (pin "b7")
-    (pin "b2")
-    (pin "b3")
-    (pin "b4")
-    (pin "b8")
-    (pin "b5")
-    (pin "b6")
-    (pin "a6")
-    (pin "b1")
-    (pin "a7")
-    (pin "b10")
-    (pin "a1")
-    (pin "b9")
-    (pin "a10")
+    (pin "1")
     (instances
       (project "BeanBoard"
         (path "/3defbfd6-25f4-40d7-986c-89ce878d27b9"
-          (reference "J13") (unit 1)
+          (reference "#PWR031") (unit 1)
         )
       )
@@
     )
   )
-  (symbol (lib_name "GND_2") (lib_id "power:GND") (at 50.8 209.55 0) (unit 1)
+  (symbol (lib_name "GND_2") (lib_id "power:GND") (at 50.8 212.09 0) (unit 1)
     (in_bom yes) (on_board yes) (dnp no)
-    (property "Reference" "#PWR032" (at 50.8 215.9 0)
+    (property "Reference" "#PWR032" (at 50.8 218.44 0)
       (effects (font (size 1.27 1.27)) hide)
     )
-    (property "Value" "GND" (at 50.8 213.36 0)
+    (property "Value" "GND" (at 50.8 215.9 0)
       (effects (font (size 1.27 1.27)))
     )
-    (property "Footprint" "" (at 50.8 209.55 0)
+    (property "Footprint" "" (at 50.8 212.09 0)
       (effects (font (size 1.27 1.27)) hide)
     )
-    (property "Datasheet" "" (at 50.8 209.55 0)
+    (property "Datasheet" "" (at 50.8 212.09 0)
       (effects (font (size 1.27 1.27)) hide)
     )
@@
         )
       )
+    )
+  )
+  (symbol (lib_id "Connector:Conn_01x10_Socket") (at 220.98 246.38 0) (unit 1)
+    (in_bom yes) (on_board yes) (dnp no)
+    (property "Reference" "J8" (at 217.17 231.14 0)
+      (effects (font (size 1.27 1.27)) (justify left))
+    )
+    (property "Value" "Conn_01x10_Socket" (at 200.66 228.6 0)
+      (effects (font (size 1.27 1.27)) (justify left) hide)
+    )
+    (property "Footprint" "Connector_PinSocket_2.54mm:PinSocket_1x10_P2.54mm_Vertical" (at 220.98 246.38 0)
+      (effects (font (size 1.27 1.27)) hide)
+    )
+    (property "Datasheet" "~" (at 220.98 246.38 0)
+      (effects (font (size 1.27 1.27)) hide)
+    )
+    (pin "9")
+    (pin "1")
+    (pin "8")
+    (pin "4")
+    (pin "2")
+    (pin "3")
+    (pin "10")
+    (pin "6")
+    (pin "7")
+    (pin "5")
+    (instances
+      (project "BeanBoard"
+        (path "/3defbfd6-25f4-40d7-986c-89ce878d27b9"
+          (reference "J8") (unit 1)
+        )
+      )

Commit message: Update BeanBoard.kicad_sch
Parts:
- J5, J6: footprint Connector_PinSocket_2.54mm:PinSocket_1x03_P2.54mm_Vertical -> Connector_PinSocket_2.54mm_alt:PinSocket_1x03_P2.54mm_Vertical_alt
Changed lines of the file:
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@@
       (effects (font (size 1.27 1.27)) (justify left))
     )
-    (property "Footprint" "Connector_PinSocket_2.54mm:PinSocket_1x03_P2.54mm_Vertical" (at 93.98 157.48 0)
+    (property "Footprint" "Connector_PinSocket_2.54mm_alt:PinSocket_1x03_P2.54mm_Vertical_alt" (at 93.98 157.48 0)
       (effects (font (size 1.27 1.27)) hide)
     )
@@
       (effects (font (size 1.27 1.27)) (justify left))
     )
-    (property "Footprint" "Connector_PinSocket_2.54mm:PinSocket_1x03_P2.54mm_Vertical" (at 93.98 146.05 0)
-      (effects (font (size 1.27 1.27)) hide)
-    )
+    (property "Footprint" "Connector_PinSocket_2.54mm_alt:PinSocket_1x03_P2.54mm_Vertical_alt" (at 93.98 146.05 0)
+      (effects (font (size 1.27 1.27)) hide)
+    )
