File: kicad/BeanBoard.kicad_sch (KiCad schematic)
At the start: 163 parts, among them J1 BZ_Address, J11 Barrel_Jack_Switch, J2 BZ_Data, J3 BZ_Control, J4 BZ_Power, J5 BZ_IORQ_enable, J6 BZ_MREQ_enable, J7 LCD, J8 Conn_01x10_Socket, J9 Conn_01x10_Socket, SW00 SW_Push_45deg, SW01 SW_Push_45deg, SW02 SW_Push_45deg, SW03 SW_Push_45deg, SW04 SW_Push_45deg, SW05 SW_Push_45deg, SW06 SW_Push_45deg, SW07 SW_Push_45deg, SW10 SW_Push_45deg, SW11 SW_Push_45deg, SW12 SW_Push_45deg, SW13 SW_Push_45deg, SW14 SW_Push_45deg, SW15 SW_Push_45deg, SW16 SW_Push_45deg, SW17 SW_Push_45deg, SW20 SW_Push_45deg, SW21 SW_Push_45deg, SW22 SW_Push_45deg, SW23 SW_Push_45deg, SW24 SW_Push_45deg, SW25 SW_Push_45deg, SW26 SW_Push_45deg, SW27 SW_Push_45deg, SW30 SW_Push_45deg, SW31 SW_Push_45deg, SW32 SW_Push_45deg, SW33 SW_Push_45deg, SW34 SW_Push_45deg, SW35 SW_Push_45deg, SW36 SW_Push_45deg, SW37 SW_Push_45deg, SW40 SW_Push_45deg, SW41 SW_Push_45deg, SW42 SW_Push_45deg, SW43 SW_Push_45deg, SW44 SW_Push_45deg, SW45 SW_Push_45deg, SW46 SW_Push_45deg, SW47 SW_Push_45deg, SW50 SW_Push_45deg, SW51 SW_Push_45deg, SW52 SW_Push_45deg, SW53 SW_Push_45deg, SW54 SW_Push_45deg, SW55 SW_Push_45deg, SW56 SW_Push_45deg, SW57 SW_Push_45deg, SW60 SW_Push_45deg, SW61 SW_Push_45deg, SW62 SW_Push_45deg, SW63 SW_Push_45deg, SW64 SW_Push_45deg, SW65 SW_Push_45deg, SW66 SW_Push_45deg, SW67 SW_Push_45deg, SW70 SW_Push_45deg, SW71 SW_Push_45deg, SW72 SW_Push_45deg, SW73 SW_Push_45deg, SW74 SW_Push_45deg, SW75 SW_Push_45deg, SW76 SW_Push_45deg, SW77 SW_Push_45deg, U1 74LS138, U2 SN74LS373, U3 74LS244, U4 SN74LS373, U5 74LS244, U6 74LS32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

Commit message: Update BeanBoard.kicad_sch
Parts:
- added J10: Address, Connector_PinSocket_2.54mm:PinSocket_1x16_P2.54mm_Vertical, symbol Connector:Conn_01x16_Socket
- added J12: Control/Data, Connector_PinSocket_2.54mm:PinSocket_1x16_P2.54mm_Vertical, symbol Connector:Conn_01x16_Socket
- added J13: Power Out, Connector_PinSocket_2.54mm:PinSocket_1x02_P2.54mm_Vertical, symbol Connector:Conn_01x02_Socket
- added JP1: MREQ_enable, Connector_PinSocket_2.54mm_alt:PinSocket_1x03_P2.54mm_Vertical_alt, symbol Jumper:Jumper_3_Bridged12
- U1: footprint Package_DIP:DIP-16_W7.62mm_Socket_LongPads -> Package_DIP:DIP-16_W7.62mm_Socket
- U2, U3, U4, U5: footprint Package_DIP:DIP-20_W7.62mm_Socket_LongPads -> Package_DIP:DIP-20_W7.62mm_Socket
- U6, U7: footprint Package_DIP:DIP-14_W7.62mm_Socket_LongPads -> Package_DIP:DIP-14_W7.62mm_Socket
Connections:
- net A0: now also J10.1 (Pin_1)
- net A1: now also J10.2 (Pin_2)
- net A10: now also J10.11 (Pin_11)
- net A11: now also J10.12 (Pin_12)
- net A12: now also J10.13 (Pin_13)
- net A13: now also J10.14 (Pin_14)
- net A14: now also J10.15 (Pin_15)
- net A15: now also J10.16 (Pin_16)
- net A2: now also J10.3 (Pin_3)
- net A3: now also J10.4 (Pin_4)
- net A4: now also J10.5 (Pin_5)
- net A5: now also J10.6 (Pin_6)
- net A6: now also J10.7 (Pin_7)
- net A7: now also J10.8 (Pin_8)
- net A8: now also J10.9 (Pin_9)
- net A9: now also J10.10 (Pin_10)
- net D0: now also J12.9 (Pin_9)
- net D1: now also J12.10 (Pin_10)
- net D2: now also J12.11 (Pin_11)
- net D3: now also J12.12 (Pin_12)
- net D4: now also J12.13 (Pin_13)
- net D5: now also J12.14 (Pin_14)
- net D6: now also J12.15 (Pin_15)
- net D7: now also J12.16 (Pin_16)
- net GND: now also J12.8 (Pin_8), J13.2 (Pin_2)
- net VCC: now also J13.1 (Pin_1)
- net ~{CLKINH}: now also J12.7 (Pin_7)
- net ~{CLK}: now also J12.6 (Pin_6)
- net ~{IORQ}: now also J12.4 (Pin_4)
- net ~{MREQ}: now also J12.3 (Pin_3)
- net ~{RD}: now also J12.1 (Pin_1)
- net ~{RESET}: now also J12.5 (Pin_5)
- net ~{WR}: now also J12.2 (Pin_2)
- net at J6.1 (Pin_1): now also JP1.1 (A); no longer J6.2 (Pin_2)
- net at J6.3 (Pin_3): now also JP1.3 (B)
- new net: J6.2 (Pin_2), JP1.2 (C)
- no-connect marks 26 -> 13
Other:
- moved on the sheet: C1, J1, J11, J2, J3, J4, J5, J6, J7, U1, U6A, U6B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

Commit message: Update BeanBoard.kicad_sch
Parts:
- J8: value Conn_01x10_Socket -> GPO
- J9: value Conn_01x10_Socket -> GPI
Connections:
- net GPI4: now reaches J9.5 (Pin_5), U5.11 (I0b)
- net GPI5: now reaches J9.6 (Pin_6), U5.13 (I1b)
- net GPI6: now reaches J9.7 (Pin_7), U5.15 (I2b)
- net GPI7: now reaches J9.8 (Pin_8), U5.17 (I3b)
- net GPI0: now reaches J9.1 (Pin_1), U5.2 (I0a)
- net GPI1: now reaches J9.2 (Pin_2), U5.4 (I1a)
- net GPI2: now reaches J9.3 (Pin_3), U5.6 (I2a)
- net GPI3: now reaches J9.4 (Pin_4), U5.8 (I3a)
- net GPO4: now reaches J8.5 (Pin_5), U4.12 (O4)
- net GPO5: now reaches J8.6 (Pin_6), U4.15 (O5)
- net GPO6: now reaches J8.7 (Pin_7), U4.16 (O6)
- net GPO7: now reaches J8.8 (Pin_8), U4.19 (O7)
- net GPO0: now reaches J8.1 (Pin_1), U4.2 (O0)
- net GPO1: now reaches J8.2 (Pin_2), U4.5 (O1)
- net GPO2: now reaches J8.3 (Pin_3), U4.6 (O2)
- net GPO3: now reaches J8.4 (Pin_4), U4.9 (O3)
Changed lines of the file:
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@@
     (effects (font (size 1.27 1.27)) (justify left bottom))
   )
+  (label "GPO0" (at 208.28 236.22 0) (fields_autoplaced)
+    (effects (font (size 1.27 1.27)) (justify left bottom))
+  )
   (label "D7" (at 173.99 254 0) (fields_autoplaced)
     (effects (font (size 1.27 1.27)) (justify left bottom))
   )
+  (label "GPI0" (at 236.22 236.22 0) (fields_autoplaced)
+    (effects (font (size 1.27 1.27)) (justify left bottom))
+  )
   (label "~{RD}" (at 189.23 154.94 180) (fields_autoplaced)
     (effects (font (size 1.27 1.27)) (justify right bottom))
@@
     (effects (font (size 1.27 1.27)) (justify right bottom))
   )
+  (label "GPO7" (at 208.28 254 0) (fields_autoplaced)
+    (effects (font (size 1.27 1.27)) (justify left bottom))
+  )
   (label "A5" (at 27.94 171.45 180) (fields_autoplaced)
     (effects (font (size 1.27 1.27)) (justify right bottom))
@@
     (effects (font (size 1.27 1.27)) (justify left bottom))
   )
+  (label "GPO1" (at 208.28 238.76 0) (fields_autoplaced)
+    (effects (font (size 1.27 1.27)) (justify left bottom))
+  )
   (label "D6" (at 276.86 251.46 0) (fields_autoplaced)
     (effects (font (size 1.27 1.27)) (justify left bottom))
@@
     (effects (font (size 1.27 1.27)) (justify left bottom))
   )
+  (label "GPO3" (at 208.28 243.84 0) (fields_autoplaced)
+    (effects (font (size 1.27 1.27)) (justify left bottom))
+  )
   (label "~{RESET}" (at 53.34 191.77 180) (fields_autoplaced)
     (effects (font (size 1.27 1.27)) (justify right bottom))
@@
     (effects (font (size 1.27 1.27)) (justify right bottom))
   )
+  (label "GPO5" (at 208.28 248.92 0) (fields_autoplaced)
+    (effects (font (size 1.27 1.27)) (justify left bottom))
+  )
   (label "GPIO_WR" (at 133.35 105.41 180) (fields_autoplaced)
     (effects (font (size 1.27 1.27)) (justify right bottom))
@@
     (effects (font (size 1.27 1.27)) (justify right bottom))
   )
+  (label "GPI2" (at 236.22 241.3 0) (fields_autoplaced)
+    (effects (font (size 1.27 1.27)) (justify left bottom))
+  )
   (label "A2" (at 16.51 36.83 0) (fields_autoplaced)
     (effects (font (size 1.27 1.27)) (justify left bottom))
@@
     (effects (font (size 1.27 1.27)) (justify left bottom))
   )
+  (label "GPI6" (at 236.22 251.46 0) (fields_autoplaced)
+    (effects (font (size 1.27 1.27)) (justify left bottom))
+  )
   (label "A12" (at 160.02 185.42 180) (fields_autoplaced)
     (effects (font (size 1.27 1.27)) (justify right bottom))
@@
     (effects (font (size 1.27 1.27)) (justify right bottom))
   )
+  (label "GPI5" (at 236.22 248.92 0) (fields_autoplaced)
+    (effects (font (size 1.27 1.27)) (justify left bottom))
+  )
   (label "A8" (at 160.02 175.26 180) (fields_autoplaced)
     (effects (font (size 1.27 1.27)) (justify right bottom))
@@
     (effects (font (size 1.27 1.27)) (justify left bottom))
   )
+  (label "GPI4" (at 236.22 246.38 0) (fields_autoplaced)
+    (effects (font (size 1.27 1.27)) (justify left bottom))
+  )
   (label "A11" (at 160.02 182.88 180) (fields_autoplaced)
     (effects (font (size 1.27 1.27)) (justify right bottom))
@@
     (effects (font (size 1.27 1.27)) (justify right bottom))
   )
+  (label "GPI7" (at 236.22 254 0) (fields_autoplaced)
+    (effects (font (size 1.27 1.27)) (justify left bottom))
+  )
   (label "D0" (at 224.79 109.22 0) (fields_autoplaced)
     (effects (font (size 1.27 1.27)) (justify left bottom))
@@
     (effects (font (size 1.27 1.27)) (justify right bottom))
   )
+  (label "GPI3" (at 236.22 243.84 0) (fields_autoplaced)
+    (effects (font (size 1.27 1.27)) (justify left bottom))
+  )
   (label "D3" (at 173.99 243.84 0) (fields_autoplaced)
     (effects (font (size 1.27 1.27)) (justify left bottom))
@@
     (effects (font (size 1.27 1.27)) (justify right bottom))
   )
+  (label "GPO4" (at 208.28 246.38 0) (fields_autoplaced)
+    (effects (font (size 1.27 1.27)) (justify left bottom))
+  )
   (label "A1" (at 27.94 161.29 180) (fields_autoplaced)
     (effects (font (size 1.27 1.27)) (justify right bottom))
@@
     (effects (font (size 1.27 1.27)) (justify left bottom))
   )
+  (label "GPI1" (at 236.22 238.76 0) (fields_autoplaced)
+    (effects (font (size 1.27 1.27)) (justify left bottom))
+  )
   (label "D7" (at 347.98 19.05 90) (fields_autoplaced)
     (effects (font (size 1.27 1.27)) (justify left bottom))
@@
     (effects (font (size 1.27 1.27)) (justify right bottom))
   )
+  (label "GPO2" (at 208.28 241.3 0) (fields_autoplaced)
+    (effects (font (size 1.27 1.27)) (justify left bottom))
+  )
   (label "D6" (at 345.44 19.05 90) (fields_autoplaced)
     (effects (font (size 1.27 1.27)) (justify left bottom))
@@
     (effects (font (size 1.27 1.27)) (justify left bottom))
   )
+  (label "GPO6" (at 208.28 251.46 0) (fields_autoplaced)
+    (effects (font (size 1.27 1.27)) (justify left bottom))
+  )
   (label "D2" (at 189.23 180.34 180) (fields_autoplaced)
     (effects (font (size 1.27 1.27)) (justify right bottom))
@@
       (effects (font (size 1.27 1.27)) (justify left))
     )
-    (property "Value" "Conn_01x10_Socket" (at 243.84 228.6 0)
+    (property "Value" "GPI" (at 243.84 228.6 0)
       (effects (font (size 1.27 1.27)) (justify left) hide)
     )
@@
       (effects (font (size 1.27 1.27)) (justify left))
     )
-    (property "Value" "Conn_01x10_Socket" (at 200.66 228.6 0)
+    (property "Value" "GPO" (at 200.66 228.6 0)
       (effects (font (size 1.27 1.27)) (justify left) hide)
     )
