File: kicad/BeanBoard.kicad_pcb (KiCad board)
At the start: 2 copper layers, 7 parts, among them J1 Address, J2 Data, J3 Control, J4 Power, J5 Reset

Commit message: Update BeanBoard.kicad_pcb
Parts:
- removed the J1 at (-14.1, 76.1)
- removed the J2 at (-100.5, 73.6)
- removed the J3 at (-14.1, 81.2)
- removed the J4 at (-100.5, 38.0)
- removed the J5 at (-82.7, 104.0)
- added C1: 0.1uF, Capacitor_THT:C_Disc_D5.0mm_W2.5mm_P2.50mm, F.Cu at (228.2, -40.2)
- added C2: 0.1uF, Capacitor_THT:C_Disc_D5.0mm_W2.5mm_P2.50mm, F.Cu at (228.2, -36.2)
- added C3: 0.1uF, Capacitor_THT:C_Disc_D5.0mm_W2.5mm_P2.50mm, F.Cu at (228.2, -32.1)
- added C4: 0.1uF, Capacitor_THT:C_Disc_D5.0mm_W2.5mm_P2.50mm, F.Cu at (228.2, -28.1)
- added C5: 0.1uF, Capacitor_THT:C_Disc_D5.0mm_W2.5mm_P2.50mm, F.Cu at (228.2, -24.1)
- added D1: 1N4148, Diode_THT:D_DO-35_SOD27_P7.62mm_Horizontal, F.Cu at (136.6, -60.0)
- added D10: 1N4148, Diode_THT:D_DO-35_SOD27_P7.62mm_Horizontal, F.Cu at (136.6, -28.1)
- added D11: 1N4148, Diode_THT:D_DO-35_SOD27_P7.62mm_Horizontal, F.Cu at (136.6, -24.5)
- added D12: 1N4148, Diode_THT:D_DO-35_SOD27_P7.62mm_Horizontal, F.Cu at (136.6, -20.9)
- added D13: 1N4148, Diode_THT:D_DO-35_SOD27_P7.62mm_Horizontal, F.Cu at (136.6, -17.4)
- added D14: 1N4148, Diode_THT:D_DO-35_SOD27_P7.62mm_Horizontal, F.Cu at (147.3, -60.0)
- added D15: 1N4148, Diode_THT:D_DO-35_SOD27_P7.62mm_Horizontal, F.Cu at (147.3, -56.5)
- added D16: 1N4148, Diode_THT:D_DO-35_SOD27_P7.62mm_Horizontal, F.Cu at (147.3, -52.9)
- added D17: 1N4148, Diode_THT:D_DO-35_SOD27_P7.62mm_Horizontal, F.Cu at (147.3, -49.4)
- added D18: 1N4148, Diode_THT:D_DO-35_SOD27_P7.62mm_Horizontal, F.Cu at (147.3, -45.8)
- added D19: 1N4148, Diode_THT:D_DO-35_SOD27_P7.62mm_Horizontal, F.Cu at (147.3, -42.2)
- added D2: 1N4148, Diode_THT:D_DO-35_SOD27_P7.62mm_Horizontal, F.Cu at (136.6, -56.5)
- added D20: 1N4148, Diode_THT:D_DO-35_SOD27_P7.62mm_Horizontal, F.Cu at (147.3, -38.7)
- added D21: 1N4148, Diode_THT:D_DO-35_SOD27_P7.62mm_Horizontal, F.Cu at (147.3, -35.1)
- added D22: 1N4148, Diode_THT:D_DO-35_SOD27_P7.62mm_Horizontal, F.Cu at (147.3, -31.6)
- added D23: 1N4148, Diode_THT:D_DO-35_SOD27_P7.62mm_Horizontal, F.Cu at (147.3, -28.1)
- added D24: 1N4148, Diode_THT:D_DO-35_SOD27_P7.62mm_Horizontal, F.Cu at (147.3, -24.5)
- added D25: 1N4148, Diode_THT:D_DO-35_SOD27_P7.62mm_Horizontal, F.Cu at (147.3, -20.9)
- added D26: 1N4148, Diode_THT:D_DO-35_SOD27_P7.62mm_Horizontal, F.Cu at (147.3, -17.4)
- added D27: 1N4148, Diode_THT:D_DO-35_SOD27_P7.62mm_Horizontal, F.Cu at (158.1, -60.0)
- added D28: 1N4148, Diode_THT:D_DO-35_SOD27_P7.62mm_Horizontal, F.Cu at (158.1, -56.5)
- added D29: 1N4148, Diode_THT:D_DO-35_SOD27_P7.62mm_Horizontal, F.Cu at (158.1, -52.9)
- added D3: 1N4148, Diode_THT:D_DO-35_SOD27_P7.62mm_Horizontal, F.Cu at (136.6, -52.9)
- added D30: 1N4148, Diode_THT:D_DO-35_SOD27_P7.62mm_Horizontal, F.Cu at (158.1, -49.4)
- added D31: 1N4148, Diode_THT:D_DO-35_SOD27_P7.62mm_Horizontal, F.Cu at (158.1, -45.8)
- added D32: 1N4148, Diode_THT:D_DO-35_SOD27_P7.62mm_Horizontal, F.Cu at (158.1, -42.2)
- added D33: 1N4148, Diode_THT:D_DO-35_SOD27_P7.62mm_Horizontal, F.Cu at (158.1, -38.7)
- added D34: 1N4148, Diode_THT:D_DO-35_SOD27_P7.62mm_Horizontal, F.Cu at (158.1, -35.1)
- added D35: 1N4148, Diode_THT:D_DO-35_SOD27_P7.62mm_Horizontal, F.Cu at (158.1, -31.6)
- added D36: 1N4148, Diode_THT:D_DO-35_SOD27_P7.62mm_Horizontal, F.Cu at (158.1, -28.1)
- added D37: 1N4148, Diode_THT:D_DO-35_SOD27_P7.62mm_Horizontal, F.Cu at (158.1, -24.5)
- added D38: 1N4148, Diode_THT:D_DO-35_SOD27_P7.62mm_Horizontal, F.Cu at (158.1, -20.9)
- added D39: 1N4148, Diode_THT:D_DO-35_SOD27_P7.62mm_Horizontal, F.Cu at (158.1, -17.4)
- added D4: 1N4148, Diode_THT:D_DO-35_SOD27_P7.62mm_Horizontal, F.Cu at (136.6, -49.4)
- added D40: 1N4148, Diode_THT:D_DO-35_SOD27_P7.62mm_Horizontal, F.Cu at (168.9, -60.0)
- added D41: 1N4148, Diode_THT:D_DO-35_SOD27_P7.62mm_Horizontal, F.Cu at (168.9, -56.5)
- added D42: 1N4148, Diode_THT:D_DO-35_SOD27_P7.62mm_Horizontal, F.Cu at (168.9, -52.9)
- added D43: 1N4148, Diode_THT:D_DO-35_SOD27_P7.62mm_Horizontal, F.Cu at (168.9, -49.4)
- added D44: 1N4148, Diode_THT:D_DO-35_SOD27_P7.62mm_Horizontal, F.Cu at (168.9, -45.8)
- added D45: 1N4148, Diode_THT:D_DO-35_SOD27_P7.62mm_Horizontal, F.Cu at (168.9, -42.2)
- added D46: 1N4148, Diode_THT:D_DO-35_SOD27_P7.62mm_Horizontal, F.Cu at (168.9, -38.7)
- added D47: 1N4148, Diode_THT:D_DO-35_SOD27_P7.62mm_Horizontal, F.Cu at (168.9, -35.1)
- added D48: 1N4148, Diode_THT:D_DO-35_SOD27_P7.62mm_Horizontal, F.Cu at (168.9, -31.6)
- added D49: 1N4148, Diode_THT:D_DO-35_SOD27_P7.62mm_Horizontal, F.Cu at (168.9, -28.1)
- added D5: 1N4148, Diode_THT:D_DO-35_SOD27_P7.62mm_Horizontal, F.Cu at (136.6, -45.8)
- added D50: 1N4148, Diode_THT:D_DO-35_SOD27_P7.62mm_Horizontal, F.Cu at (168.9, -24.5)
- added D51: 1N4148, Diode_THT:D_DO-35_SOD27_P7.62mm_Horizontal, F.Cu at (168.9, -20.9)
- added D52: 1N4148, Diode_THT:D_DO-35_SOD27_P7.62mm_Horizontal, F.Cu at (168.9, -17.4)
- added D53: 1N4148, Diode_THT:D_DO-35_SOD27_P7.62mm_Horizontal, F.Cu at (179.6, -60.0)
- added D54: 1N4148, Diode_THT:D_DO-35_SOD27_P7.62mm_Horizontal, F.Cu at (179.6, -56.5)
- added D55: 1N4148, Diode_THT:D_DO-35_SOD27_P7.62mm_Horizontal, F.Cu at (179.6, -52.9)
- added D56: 1N4148, Diode_THT:D_DO-35_SOD27_P7.62mm_Horizontal, F.Cu at (179.6, -49.4)
- added D57: 1N4148, Diode_THT:D_DO-35_SOD27_P7.62mm_Horizontal, F.Cu at (179.6, -45.8)
- added D58: 1N4148, Diode_THT:D_DO-35_SOD27_P7.62mm_Horizontal, F.Cu at (179.6, -42.2)
- added D59: 1N4148, Diode_THT:D_DO-35_SOD27_P7.62mm_Horizontal, F.Cu at (179.6, -38.7)
- added D6: 1N4148, Diode_THT:D_DO-35_SOD27_P7.62mm_Horizontal, F.Cu at (136.6, -42.2)
- added D60: 1N4148, Diode_THT:D_DO-35_SOD27_P7.62mm_Horizontal, F.Cu at (179.6, -35.1)
- added D61: 1N4148, Diode_THT:D_DO-35_SOD27_P7.62mm_Horizontal, F.Cu at (179.6, -31.6)
- added D62: 1N4148, Diode_THT:D_DO-35_SOD27_P7.62mm_Horizontal, F.Cu at (179.6, -28.1)
- added D63: 1N4148, Diode_THT:D_DO-35_SOD27_P7.62mm_Horizontal, F.Cu at (179.6, -24.5)
- added D64: 1N4148, Diode_THT:D_DO-35_SOD27_P7.62mm_Horizontal, F.Cu at (179.6, -20.9)
- added D7: 1N4148, Diode_THT:D_DO-35_SOD27_P7.62mm_Horizontal, F.Cu at (136.6, -38.7)
- added D8: 1N4148, Diode_THT:D_DO-35_SOD27_P7.62mm_Horizontal, F.Cu at (136.6, -35.1)
- added D9: 1N4148, Diode_THT:D_DO-35_SOD27_P7.62mm_Horizontal, F.Cu at (136.6, -31.6)
- added J1: Address, Connector_PinSocket_2.54mm:PinSocket_1x16_P2.54mm_Vertical, F.Cu at (126.6, 92.3)
- added J1: BZ_Address, Connector_PinSocket_2.54mm:PinSocket_1x16_P2.54mm_Vertical, F.Cu at (65.4, -100.9)
- added J2: BZ_Data, Connector_PinSocket_2.54mm:PinSocket_1x08_P2.54mm_Vertical, F.Cu at (89.4, -165.2)
- added J2: Data, Connector_PinSocket_2.54mm:PinSocket_1x08_P2.54mm_Vertical, F.Cu at (40.3, 89.7)
- added J3: Control, Connector_PinSocket_2.54mm:PinSocket_1x07_P2.54mm_Vertical, F.Cu at (126.6, 97.3)
- added J3: BZ_Control, Connector_PinSocket_2.54mm:PinSocket_1x07_P2.54mm_Vertical, F.Cu at (82.4, -72.5)
- added J4: Power, Connector_PinSocket_2.54mm:PinSocket_1x02_P2.54mm_Vertical, F.Cu at (40.3, 54.2)
- added J4: BZ_Power, Connector_PinSocket_2.54mm:PinSocket_1x02_P2.54mm_Vertical, F.Cu at (63.4, -158.3)
- added J5: Reset, Connector_PinSocket_2.54mm:PinSocket_1x02_P2.54mm_Vertical, F.Cu at (58.0, 120.2)
- added J5: BZ_IORQ_enable, Connector_PinSocket_2.54mm:PinSocket_1x03_P2.54mm_Vertical, F.Cu at (52.0, -37.7)
- added J6: BZ_MREQ_enable, Connector_PinSocket_2.54mm:PinSocket_1x03_P2.54mm_Vertical, F.Cu at (70.6, -44.6)
- added J7: LCD, Connector_PinSocket_2.54mm:PinSocket_1x16_P2.54mm_Vertical, F.Cu at (295.1, -113.6)
- added R1: 10k, Resistor_THT:R_Axial_DIN0204_L3.6mm_D1.6mm_P7.62mm_Horizontal, F.Cu at (246.5, -60.2)
- added R2: 10k, Resistor_THT:R_Axial_DIN0204_L3.6mm_D1.6mm_P7.62mm_Horizontal, F.Cu at (246.5, -57.0)
- added R3: 10k, Resistor_THT:R_Axial_DIN0204_L3.6mm_D1.6mm_P7.62mm_Horizontal, F.Cu at (246.5, -53.9)
- added R4: 10k, Resistor_THT:R_Axial_DIN0204_L3.6mm_D1.6mm_P7.62mm_Horizontal, F.Cu at (246.5, -50.8)
- added R5: 10k, Resistor_THT:R_Axial_DIN0204_L3.6mm_D1.6mm_P7.62mm_Horizontal, F.Cu at (246.5, -47.6)
- added R6: 10k, Resistor_THT:R_Axial_DIN0204_L3.6mm_D1.6mm_P7.62mm_Horizontal, F.Cu at (246.5, -44.5)
- added R7: 10k, Resistor_THT:R_Axial_DIN0204_L3.6mm_D1.6mm_P7.62mm_Horizontal, F.Cu at (246.5, -41.3)
- added R8: 10k, Resistor_THT:R_Axial_DIN0204_L3.6mm_D1.6mm_P7.62mm_Horizontal, F.Cu at (246.5, -38.1)
- added R9: 220R, Resistor_THT:R_Axial_DIN0204_L3.6mm_D1.6mm_P7.62mm_Horizontal, F.Cu at (246.5, -35.0)
- added RV1: 50k, Connector_PinSocket_2.54mm:PinSocket_1x03_P2.54mm_Vertical, F.Cu at (294.5, -152.0)
- added S12: SW_Push_45deg, SW_B3F-4000_OMR:SW_B3F-4000_OMR, F.Cu at (136.7, -177.3)
- added S21: SW_Push_45deg, SW_B3F-4000_OMR:SW_B3F-4000_OMR, F.Cu at (136.7, -162.1)
- added SW00: SW_Push_45deg, SW_B3F-4000_OMR:SW_B3F-4000_OMR, F.Cu at (136.7, -146.9)
- added SW01: SW_Push_45deg, SW_B3F-4000_OMR:SW_B3F-4000_OMR, F.Cu at (136.7, -131.8)
- added SW02: SW_Push_45deg, SW_B3F-4000_OMR:SW_B3F-4000_OMR, F.Cu at (136.7, -116.6)
- added SW03: SW_Push_45deg, SW_B3F-4000_OMR:SW_B3F-4000_OMR, F.Cu at (136.7, -101.4)
- added SW04: SW_Push_45deg, SW_B3F-4000_OMR:SW_B3F-4000_OMR, F.Cu at (136.7, -86.3)
- added SW05: SW_Push_45deg, SW_B3F-4000_OMR:SW_B3F-4000_OMR, F.Cu at (136.7, -71.1)
- added SW06: SW_Push_45deg, SW_B3F-4000_OMR:SW_B3F-4000_OMR, F.Cu at (152.5, -177.3)
- added SW07: SW_Push_45deg, SW_B3F-4000_OMR:SW_B3F-4000_OMR, F.Cu at (152.5, -162.1)
- added SW10: SW_Push_45deg, SW_B3F-4000_OMR:SW_B3F-4000_OMR, F.Cu at (152.5, -146.9)
- added SW11: SW_Push_45deg, SW_B3F-4000_OMR:SW_B3F-4000_OMR, F.Cu at (152.5, -131.8)
- added SW13: SW_Push_45deg, SW_B3F-4000_OMR:SW_B3F-4000_OMR, F.Cu at (152.5, -116.6)
- added SW14: SW_Push_45deg, SW_B3F-4000_OMR:SW_B3F-4000_OMR, F.Cu at (152.5, -101.4)
- added SW15: SW_Push_45deg, SW_B3F-4000_OMR:SW_B3F-4000_OMR, F.Cu at (152.5, -86.3)
- added SW16: SW_Push_45deg, SW_B3F-4000_OMR:SW_B3F-4000_OMR, F.Cu at (152.5, -71.1)
- added SW17: SW_Push_45deg, SW_B3F-4000_OMR:SW_B3F-4000_OMR, F.Cu at (168.4, -177.3)
- added SW20: SW_Push_45deg, SW_B3F-4000_OMR:SW_B3F-4000_OMR, F.Cu at (168.4, -162.1)
- added SW22: SW_Push_45deg, SW_B3F-4000_OMR:SW_B3F-4000_OMR, F.Cu at (168.4, -146.9)
- added SW23: SW_Push_45deg, SW_B3F-4000_OMR:SW_B3F-4000_OMR, F.Cu at (168.4, -131.8)
- added SW24: SW_Push_45deg, SW_B3F-4000_OMR:SW_B3F-4000_OMR, F.Cu at (168.4, -116.6)
- added SW25: SW_Push_45deg, SW_B3F-4000_OMR:SW_B3F-4000_OMR, F.Cu at (168.4, -101.4)
- added SW26: SW_Push_45deg, SW_B3F-4000_OMR:SW_B3F-4000_OMR, F.Cu at (168.4, -86.3)
- added SW27: SW_Push_45deg, SW_B3F-4000_OMR:SW_B3F-4000_OMR, F.Cu at (168.4, -71.1)
- added SW30: SW_Push_45deg, SW_B3F-4000_OMR:SW_B3F-4000_OMR, F.Cu at (184.3, -177.3)
- added SW31: SW_Push_45deg, SW_B3F-4000_OMR:SW_B3F-4000_OMR, F.Cu at (184.3, -162.1)
- added SW32: SW_Push_45deg, SW_B3F-4000_OMR:SW_B3F-4000_OMR, F.Cu at (184.3, -146.9)
- added SW33: SW_Push_45deg, SW_B3F-4000_OMR:SW_B3F-4000_OMR, F.Cu at (184.3, -131.8)
- added SW34: SW_Push_45deg, SW_B3F-4000_OMR:SW_B3F-4000_OMR, F.Cu at (184.3, -116.6)
- added SW37: SW_Push_45deg, SW_B3F-4000_OMR:SW_B3F-4000_OMR, F.Cu at (184.3, -101.4)
- added SW40: SW_Push_45deg, SW_B3F-4000_OMR:SW_B3F-4000_OMR, F.Cu at (184.3, -86.3)
- added SW41: SW_Push_45deg, SW_B3F-4000_OMR:SW_B3F-4000_OMR, F.Cu at (184.3, -71.1)
- added SW42: SW_Push_45deg, SW_B3F-4000_OMR:SW_B3F-4000_OMR, F.Cu at (200.1, -177.3)
- added SW43: SW_Push_45deg, SW_B3F-4000_OMR:SW_B3F-4000_OMR, F.Cu at (200.1, -162.1)
- added SW44: SW_Push_45deg, SW_B3F-4000_OMR:SW_B3F-4000_OMR, F.Cu at (200.1, -146.9)
- added SW45: SW_Push_45deg, SW_B3F-4000_OMR:SW_B3F-4000_OMR, F.Cu at (200.1, -131.8)
- added SW47: SW_Push_45deg, SW_B3F-4000_OMR:SW_B3F-4000_OMR, F.Cu at (200.1, -116.6)
- added SW50: SW_Push_45deg, SW_B3F-4000_OMR:SW_B3F-4000_OMR, F.Cu at (200.1, -101.4)
- added SW51: SW_Push_45deg, SW_B3F-4000_OMR:SW_B3F-4000_OMR, F.Cu at (200.1, -86.3)
- added SW52: SW_Push_45deg, SW_B3F-4000_OMR:SW_B3F-4000_OMR, F.Cu at (200.1, -71.1)
- added SW53: SW_Push_45deg, SW_B3F-4000_OMR:SW_B3F-4000_OMR, F.Cu at (216.0, -177.3)
- added SW54: SW_Push_45deg, SW_B3F-4000_OMR:SW_B3F-4000_OMR, F.Cu at (216.0, -162.1)
- added SW55: SW_Push_45deg, SW_B3F-4000_OMR:SW_B3F-4000_OMR, F.Cu at (216.0, -146.9)
- added SW56: SW_Push_45deg, SW_B3F-4000_OMR:SW_B3F-4000_OMR, F.Cu at (216.0, -131.8)
- added SW57: SW_Push_45deg, SW_B3F-4000_OMR:SW_B3F-4000_OMR, F.Cu at (216.0, -116.6)
- added SW60: SW_Push_45deg, SW_B3F-4000_OMR:SW_B3F-4000_OMR, F.Cu at (216.0, -101.4)
- added SW61: SW_Push_45deg, SW_B3F-4000_OMR:SW_B3F-4000_OMR, F.Cu at (216.0, -86.3)
- added SW62: SW_Push_45deg, SW_B3F-4000_OMR:SW_B3F-4000_OMR, F.Cu at (216.0, -71.1)
- added SW63: SW_Push_45deg, SW_B3F-4000_OMR:SW_B3F-4000_OMR, F.Cu at (231.9, -177.3)
- added SW64: SW_Push_45deg, SW_B3F-4000_OMR:SW_B3F-4000_OMR, F.Cu at (231.9, -162.1)
- added SW65: SW_Push_45deg, SW_B3F-4000_OMR:SW_B3F-4000_OMR, F.Cu at (231.9, -146.9)
- added SW66: SW_Push_45deg, SW_B3F-4000_OMR:SW_B3F-4000_OMR, F.Cu at (231.9, -131.8)
- added SW67: SW_Push_45deg, SW_B3F-4000_OMR:SW_B3F-4000_OMR, F.Cu at (231.9, -116.6)
- added SW70: SW_Push_45deg, SW_B3F-4000_OMR:SW_B3F-4000_OMR, F.Cu at (231.9, -101.4)
- added SW71: SW_Push_45deg, SW_B3F-4000_OMR:SW_B3F-4000_OMR, F.Cu at (231.9, -86.3)
- added SW72: SW_Push_45deg, SW_B3F-4000_OMR:SW_B3F-4000_OMR, F.Cu at (231.9, -71.1)
- added SW73: SW_Push_45deg, SW_B3F-4000_OMR:SW_B3F-4000_OMR, F.Cu at (247.7, -177.3)
- added SW74: SW_Push_45deg, SW_B3F-4000_OMR:SW_B3F-4000_OMR, F.Cu at (247.7, -162.1)
- added SW75: SW_Push_45deg, SW_B3F-4000_OMR:SW_B3F-4000_OMR, F.Cu at (247.7, -146.9)
- added SW76: SW_Push_45deg, SW_B3F-4000_OMR:SW_B3F-4000_OMR, F.Cu at (247.7, -131.8)
- added SW77: SW_Push_45deg, SW_B3F-4000_OMR:SW_B3F-4000_OMR, F.Cu at (247.7, -116.6)
- added SWC46: SW_Push_45deg, SW_B3F-4000_OMR:SW_B3F-4000_OMR, F.Cu at (247.7, -101.4)
- added SWD35: SW_Push_45deg, SW_B3F-4000_OMR:SW_B3F-4000_OMR, F.Cu at (247.7, -86.3)
- added SWX36: SW_Push_45deg, SW_B3F-4000_OMR:SW_B3F-4000_OMR, F.Cu at (247.7, -71.1)
- added U1: 74LS32, Package_DIP:DIP-14_W7.62mm_Socket_LongPads, F.Cu at (214.4, -59.6)
- added U2: 74LS04, Package_DIP:DIP-14_W7.62mm_Socket_LongPads, F.Cu at (226.2, -59.6)
- added U4: 74LS138, Package_DIP:DIP-16_W7.62mm_Socket_LongPads, F.Cu at (257.7, -59.6)
- added U5: SN74LS373, Package_DIP:DIP-20_W7.62mm_Socket_LongPads, F.Cu at (190.9, -59.6)
- added U6: 74LS244, Package_DIP:DIP-20_W7.62mm_Socket_LongPads, F.Cu at (202.7, -59.6)
- moved JP1 141.7 mm to (106.3, 117.7)
- moved JP2 141.7 mm to (93.6, 117.7)
Connections:
- JP1 pad 1: (no net) -> /~{IORQ}
- JP1 pad 3: (no net) -> VCC
- JP2 pad 1: (no net) -> /~{MREQ}
- JP2 pad 3: (no net) -> VCC
Other:
- board text added: "PainfulDiodes BeanZee"
- board text removed: "BeanZee"

Commit message: Update BeanBoard.kicad_pcb
Parts:
- removed the J1 at (126.6, 92.3)
- removed the J2 at (40.3, 89.7)
- removed the J3 at (126.6, 97.3)
- removed the J4 at (40.3, 54.2)
- removed JP1: IORQ_enable, Connector_PinHeader_2.54mm:PinHeader_1x03_P2.54mm_Vertical
- removed JP2: MREQ_enable, Connector_PinHeader_2.54mm:PinHeader_1x03_P2.54mm_Vertical
- moved J2 259.6 mm to (40.3, 89.7)
- moved J4 213.7 mm to (40.3, 54.2)
- moved J1 202.7 mm to (126.6, 92.3), turned to 180 degrees
- moved J3 175.5 mm to (126.6, 97.3)
- moved J5 164.6 mm to (106.3, 117.7), turned to 90 degrees
- moved J6 163.8 mm to (93.6, 117.7), turned to 90 degrees

Commit message: Update BeanBoard.kicad_pcb
Parts:
- moved C1 194.4 mm to (37.1, -4.00)
- moved RV1 181.9 mm to (260.7, 26.8)
- moved J7 173.0 mm to (200.3, 31.1), turned to 90 degrees
- moved U5 168.4 mm to (34.9, 3.88)
- moved U1 140.3 mm to (89.5, 4.20)
- moved C3 139.0 mm to (92.3, -3.01)
- moved R1 134.1 mm to (163.5, 45.1)
- moved R2 134.1 mm to (163.5, 48.3)
- moved R3 134.1 mm to (163.5, 51.5)
- moved R4 134.1 mm to (163.5, 54.6)
- moved R5 134.1 mm to (163.5, 57.8)
- moved R6 134.1 mm to (163.5, 60.9)
- moved R7 134.1 mm to (163.5, 64.0)
- moved R8 134.1 mm to (163.5, 67.2)
- moved R9 134.1 mm to (163.5, 70.3)
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
Commit message: Update BeanBoard.kicad_pcb
Reset
Parts:
- removed D1, D18, D19, D2, D28, D29, D3, D38, D39, D4, D48, D49, D5, D58, D59, D6, D7, D8, D9: 1N4148, Diode_THT:D_DO-35_SOD27_P7.62mm_Horizontal
- removed the J5 at (58.0, 120.2)
- removed the J5 at (106.3, 117.7)
- removed S12, S21, SWC46, SWD35, SWX36: SW_Push_45deg, SW_B3F-4000_OMR:SW_B3F-4000_OMR
- added C6: 0.1uF, Capacitor_THT:C_Disc_D5.0mm_W2.5mm_P2.50mm, F.Cu at (277.6, -139.8)
- added C7: 0.1uF, Capacitor_THT:C_Disc_D5.0mm_W2.5mm_P2.50mm, F.Cu at (277.6, -135.8)
- added D00: 1N4148, Diode_THT:D_DO-35_SOD27_P7.62mm_Horizontal, F.Cu at (150.2, -67.3)
- added D01: 1N4148, Diode_THT:D_DO-35_SOD27_P7.62mm_Horizontal, F.Cu at (150.2, -63.8)
- added D02: 1N4148, Diode_THT:D_DO-35_SOD27_P7.62mm_Horizontal, F.Cu at (150.2, -60.2)
- added D03: 1N4148, Diode_THT:D_DO-35_SOD27_P7.62mm_Horizontal, F.Cu at (150.2, -56.7)
- added D04: 1N4148, Diode_THT:D_DO-35_SOD27_P7.62mm_Horizontal, F.Cu at (150.2, -53.1)
- added D05: 1N4148, Diode_THT:D_DO-35_SOD27_P7.62mm_Horizontal, F.Cu at (150.2, -49.6)
- added D06: 1N4148, Diode_THT:D_DO-35_SOD27_P7.62mm_Horizontal, F.Cu at (150.2, -46.0)
- added D07: 1N4148, Diode_THT:D_DO-35_SOD27_P7.62mm_Horizontal, F.Cu at (150.2, -42.5)
- added D65: 1N4148, Diode_THT:D_DO-35_SOD27_P7.62mm_Horizontal, F.Cu at (193.3, -63.8)
- added D66: 1N4148, Diode_THT:D_DO-35_SOD27_P7.62mm_Horizontal, F.Cu at (193.3, -60.2)
- added D67: 1N4148, Diode_THT:D_DO-35_SOD27_P7.62mm_Horizontal, F.Cu at (193.3, -56.7)
- added D70: 1N4148, Diode_THT:D_DO-35_SOD27_P7.62mm_Horizontal, F.Cu at (193.3, -53.1)
- added D71: 1N4148, Diode_THT:D_DO-35_SOD27_P7.62mm_Horizontal, F.Cu at (193.3, -49.6)
- added D72: 1N4148, Diode_THT:D_DO-35_SOD27_P7.62mm_Horizontal, F.Cu at (193.3, -46.0)
- added D73: 1N4148, Diode_THT:D_DO-35_SOD27_P7.62mm_Horizontal, F.Cu at (193.3, -42.5)
- added D74: 1N4148, Diode_THT:D_DO-35_SOD27_P7.62mm_Horizontal, F.Cu at (193.3, -38.9)
- added D75: 1N4148, Diode_THT:D_DO-35_SOD27_P7.62mm_Horizontal, F.Cu at (193.3, -35.4)
- added D76: 1N4148, Diode_THT:D_DO-35_SOD27_P7.62mm_Horizontal, F.Cu at (193.3, -31.8)
- added D77: 1N4148, Diode_THT:D_DO-35_SOD27_P7.62mm_Horizontal, F.Cu at (193.3, -28.3)
- added J5: BZ_IORQ_enable, Connector_PinSocket_2.54mm:PinSocket_1x07_P2.54mm_Vertical, F.Cu at (279.4, -47.3)
- added J8: GPO, Connector_PinSocket_2.54mm:PinSocket_1x08_P2.54mm_Vertical, F.Cu at (265.6, -47.3)
- added J9: GPI, Connector_PinSocket_2.54mm:PinSocket_1x08_P2.54mm_Vertical, F.Cu at (270.2, -47.3)
- added SW12: SW_Push_45deg, SW_B3F-4000_OMR:SW_B3F-4000_OMR, F.Cu at (166.2, -154.3)
- added SW21: SW_Push_45deg, SW_B3F-4000_OMR:SW_B3F-4000_OMR, F.Cu at (182.0, -169.4)
- added SW35: SW_Push_45deg, SW_B3F-4000_OMR:SW_B3F-4000_OMR, F.Cu at (197.9, -108.8)
- added SW36: SW_Push_45deg, SW_B3F-4000_OMR:SW_B3F-4000_OMR, F.Cu at (197.9, -93.6)
- added SW46: SW_Push_45deg, SW_B3F-4000_OMR:SW_B3F-4000_OMR, F.Cu at (213.8, -93.6)
- added U3: 74LS244, Package_DIP:DIP-20_W7.62mm_Socket_LongPads, F.Cu at (216.3, -67.0)
- added U7: 74LS04, Package_DIP:DIP-14_W7.62mm_Socket_LongPads, F.Cu at (272.5, -67.0)
- J6: footprint Connector_PinSocket_2.54mm:PinSocket_1x03_P2.54mm_Vertical -> Connector_PinSocket_2.54mm:PinSocket_1x07_P2.54mm_Vertical
- U1: value 74LS32 -> 74LS138; footprint Package_DIP:DIP-14_W7.62mm_Socket_LongPads -> Package_DIP:DIP-16_W7.62mm_Socket_LongPads
- U2: value 74LS04 -> SN74LS373; footprint Package_DIP:DIP-14_W7.62mm_Socket_LongPads -> Package_DIP:DIP-20_W7.62mm_Socket_LongPads
- U4: value 74LS138 -> SN74LS373; footprint Package_DIP:DIP-16_W7.62mm_Socket_LongPads -> Package_DIP:DIP-20_W7.62mm_Socket_LongPads
- U5: value SN74LS373 -> 74LS244
- U6: value 74LS244 -> 74LS32; footprint Package_DIP:DIP-20_W7.62mm_Socket_LongPads -> Package_DIP:DIP-14_W7.62mm_Socket_LongPads
- moved J4 292.2 mm to (282.5, -109.3)
- moved C1 286.6 mm to (277.6, -160.1)
- moved R1 260.1 mm to (277.0, -188.8)
- moved R2 260.1 mm to (277.0, -185.7)
- moved R3 260.1 mm to (277.0, -182.6)
- moved R4 260.1 mm to (277.0, -179.4)
- moved R5 260.1 mm to (277.0, -176.2)
- moved R6 260.1 mm to (277.0, -173.1)
- moved R7 260.1 mm to (277.0, -169.9)
- moved R8 260.1 mm to (277.0, -166.8)
- moved R9 260.1 mm to (277.0, -163.7)
- moved J2 259.8 mm to (261.0, -47.3)
- moved J6 251.9 mm to (284.0, -47.3), turned to 0 degrees
- moved C3 237.7 mm to (277.6, -151.9)
- moved U1 232.0 mm to (277.6, -131.6)
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Connections:
- D10 pad 1: Net-(D10-K) -> Net-(D00-K)
- D11 pad 1: Net-(D11-K) -> Net-(D01-K)
- D12 pad 1: Net-(D12-K) -> Net-(D02-K)
- D13 pad 1: Net-(D10-K) -> Net-(D03-K)
- D14 pad 1: Net-(D11-K) -> Net-(D04-K)
- D15 pad 1: Net-(D15-K) -> Net-(D05-K)
- D16 pad 1: Net-(D15-K) -> Net-(D06-K)
- D17 pad 1: Net-(D15-K) -> Net-(D07-K)
- D20 pad 1: Net-(D15-K) -> Net-(D00-K)
- D21 pad 1: Net-(D15-K) -> Net-(D01-K)
- D22 pad 1: Net-(D15-K) -> Net-(D02-K)
- D23 pad 1: Net-(D12-K) -> Net-(D03-K)
- D24 pad 1: Net-(D10-K) -> Net-(D04-K)
- D25 pad 1: Net-(D11-K) -> Net-(D05-K)
- D26 pad 1: Net-(D12-K) -> Net-(D06-K)
- D27 pad 1: Net-(D10-K) -> Net-(D07-K)
- D30 pad 1: Net-(D29-K) -> Net-(D00-K)
- D31 pad 1: Net-(D29-K) -> Net-(D01-K)
- D32 pad 1: Net-(D29-K) -> Net-(D02-K)
- D33 pad 1: Net-(D29-K) -> Net-(D03-K)
- D34 pad 1: Net-(D29-K) -> Net-(D04-K)
- D35 pad 1: Net-(D29-K) -> Net-(D05-K)
- D36 pad 1: Net-(D29-K) -> Net-(D06-K)
- D37 pad 1: Net-(D12-K) -> Net-(D07-K)
- D40 pad 1: Net-(D12-K) -> Net-(D00-K)
- D41 pad 1: Net-(D10-K) -> Net-(D01-K)
- D42 pad 1: Net-(D11-K) -> Net-(D02-K)
- D43 pad 1: Net-(D43-K) -> Net-(D03-K)
- D44 pad 1: Net-(D43-K) -> Net-(D04-K)
- D45 pad 1: Net-(D43-K) -> Net-(D05-K)
- D46 pad 1: Net-(D43-K) -> Net-(D06-K)
- D47 pad 1: Net-(D43-K) -> Net-(D07-K)
- D50 pad 1: Net-(D43-K) -> Net-(D00-K)
- D51 pad 1: Net-(D12-K) -> Net-(D01-K)
- D52 pad 1: Net-(D10-K) -> Net-(D02-K)
- D53 pad 1: Net-(D11-K) -> Net-(D03-K)
- D54 pad 1: Net-(D12-K) -> Net-(D04-K)
- D55 pad 1: Net-(D10-K) -> Net-(D05-K)
- D56 pad 1: Net-(D11-K) -> Net-(D06-K)
- D57 pad 1: Net-(D57-K) -> Net-(D07-K)
- D60 pad 1: Net-(D57-K) -> Net-(D00-K)
- D61 pad 1: Net-(D57-K) -> Net-(D01-K)
- D62 pad 1: Net-(D57-K) -> Net-(D02-K)
- D63 pad 1: Net-(D57-K) -> Net-(D03-K)
- D64 pad 1: Net-(D57-K) -> Net-(D04-K)
- J7 pad 5: /LCD_R/~{W} -> /RD
- R1 pad 2: Net-(D1-K) -> Net-(D00-K)
- R2 pad 2: Net-(D15-K) -> Net-(D01-K)
- R3 pad 2: Net-(D29-K) -> Net-(D02-K)
- R4 pad 2: Net-(D43-K) -> Net-(D03-K)
- R5 pad 2: Net-(D57-K) -> Net-(D04-K)
- R6 pad 2: Net-(D12-K) -> Net-(D05-K)
- R7 pad 2: Net-(D10-K) -> Net-(D06-K)
- R8 pad 2: Net-(D11-K) -> Net-(D07-K)
- SW00 pad 1: Net-(U5-O0) -> Net-(U2-O0)
- SW01 pad 1: Net-(U5-O0) -> Net-(U2-O0)
- SW01 pad 2: Net-(D15-A) -> Net-(D01-A)
- SW02 pad 1: Net-(U5-O0) -> Net-(U2-O0)
- SW03 pad 1: Net-(U5-O0) -> Net-(U2-O0)
- SW03 pad 2: Net-(D43-A) -> Net-(D03-A)
- SW04 pad 1: Net-(U5-O0) -> Net-(U2-O0)
- SW04 pad 2: Net-(D57-A) -> Net-(D04-A)
- SW05 pad 1: Net-(U5-O0) -> Net-(U2-O0)
- SW06 pad 1: Net-(U5-O0) -> Net-(U2-O0)
- SW06 pad 2: Net-(D10-A) -> Net-(D06-A)
- SW07 pad 1: Net-(U5-O0) -> Net-(U2-O0)
- SW07 pad 2: Net-(D11-A) -> Net-(D07-A)
- SW10 pad 1: Net-(U5-O1) -> Net-(U2-O1)
- SW10 pad 2: Net-(D2-A) -> Net-(D10-A)
- SW11 pad 1: Net-(U5-O1) -> Net-(U2-O1)
- SW11 pad 2: Net-(D16-A) -> Net-(D11-A)
- SW13 pad 1: Net-(U5-O1) -> Net-(U2-O1)
- SW13 pad 2: Net-(D44-A) -> Net-(D13-A)
- SW14 pad 1: Net-(U5-O1) -> Net-(U2-O1)
- SW14 pad 2: Net-(D58-A) -> Net-(D14-A)
- SW15 pad 1: Net-(U5-O1) -> Net-(U2-O1)
- SW15 pad 2: Net-(D12-A) -> Net-(D15-A)
- SW16 pad 1: Net-(U5-O1) -> Net-(U2-O1)
- SW16 pad 2: Net-(D13-A) -> Net-(D16-A)
- SW17 pad 1: Net-(U5-O1) -> Net-(U2-O1)
- SW17 pad 2: Net-(D14-A) -> Net-(D17-A)
- SW20 pad 1: Net-(U5-O2) -> Net-(U2-O2)
- SW20 pad 2: Net-(D3-A) -> Net-(D20-A)
- SW22 pad 1: Net-(U5-O2) -> Net-(U2-O2)
- SW22 pad 2: Net-(D31-A) -> Net-(D22-A)
- SW23 pad 1: Net-(U5-O2) -> Net-(U2-O2)
- SW23 pad 2: Net-(D45-A) -> Net-(D23-A)
- SW24 pad 1: Net-(U5-O2) -> Net-(U2-O2)
- SW24 pad 2: Net-(D59-A) -> Net-(D24-A)
- SW25 pad 1: Net-(U5-O2) -> Net-(U2-O2)
- SW25 pad 2: Net-(D23-A) -> Net-(D25-A)
- SW26 pad 1: Net-(U5-O2) -> Net-(U2-O2)
- SW26 pad 2: Net-(D24-A) -> Net-(D26-A)
- SW27 pad 1: Net-(U5-O2) -> Net-(U2-O2)
- SW27 pad 2: Net-(D25-A) -> Net-(D27-A)
- SW30 pad 1: Net-(U5-O3) -> Net-(U2-O3)
- SW30 pad 2: Net-(D4-A) -> Net-(D30-A)
- SW31 pad 1: Net-(U5-O3) -> Net-(U2-O3)
- SW31 pad 2: Net-(D18-A) -> Net-(D31-A)
- SW32 pad 1: Net-(U5-O3) -> Net-(U2-O3)
- SW33 pad 1: Net-(U5-O3) -> Net-(U2-O3)
- SW33 pad 2: Net-(D46-A) -> Net-(D33-A)
- SW34 pad 1: Net-(U5-O3) -> Net-(U2-O3)
- SW34 pad 2: Net-(D60-A) -> Net-(D34-A)
- SW37 pad 1: Net-(U5-O3) -> Net-(U2-O3)
- SW37 pad 2: Net-(D28-A) -> Net-(D37-A)
- SW40 pad 1: Net-(U5-O4) -> Net-(U2-O4)
- SW40 pad 2: Net-(D5-A) -> Net-(D40-A)
- SW41 pad 1: Net-(U5-O4) -> Net-(U2-O4)
- SW41 pad 2: Net-(D19-A) -> Net-(D41-A)
- SW42 pad 1: Net-(U5-O4) -> Net-(U2-O4)
- SW42 pad 2: Net-(D33-A) -> Net-(D42-A)
- SW43 pad 1: Net-(U5-O4) -> Net-(U2-O4)
- SW43 pad 2: Net-(D47-A) -> Net-(D43-A)
- SW44 pad 1: Net-(U5-O4) -> Net-(U2-O4)
- SW44 pad 2: Net-(D61-A) -> Net-(D44-A)
- SW45 pad 1: Net-(U5-O4) -> Net-(U2-O4)
- SW45 pad 2: Net-(D37-A) -> Net-(D45-A)
- SW47 pad 1: Net-(U5-O4) -> Net-(U2-O4)
- SW47 pad 2: Net-(D39-A) -> Net-(D47-A)
- SW50 pad 1: Net-(U5-O5) -> Net-(U2-O5)
- SW50 pad 2: Net-(D6-A) -> Net-(D50-A)
- SW51 pad 1: Net-(U5-O5) -> Net-(U2-O5)
- SW51 pad 2: Net-(D20-A) -> Net-(D51-A)
- SW52 pad 1: Net-(U5-O5) -> Net-(U2-O5)
- SW52 pad 2: Net-(D34-A) -> Net-(D52-A)
- SW53 pad 1: Net-(U5-O5) -> Net-(U2-O5)
- SW53 pad 2: Net-(D48-A) -> Net-(D53-A)
- SW54 pad 1: Net-(U5-O5) -> Net-(U2-O5)
- SW54 pad 2: Net-(D62-A) -> Net-(D54-A)
- SW55 pad 1: Net-(U5-O5) -> Net-(U2-O5)
- SW55 pad 2: Net-(D40-A) -> Net-(D55-A)
- SW56 pad 1: Net-(U5-O5) -> Net-(U2-O5)
- SW56 pad 2: Net-(D41-A) -> Net-(D56-A)
- SW57 pad 1: Net-(U5-O5) -> Net-(U2-O5)
- SW57 pad 2: Net-(D42-A) -> Net-(D57-A)
- SW60 pad 1: Net-(U5-O6) -> Net-(U2-O6)
- SW60 pad 2: Net-(D7-A) -> Net-(D60-A)
- SW61 pad 1: Net-(U5-O6) -> Net-(U2-O6)
- SW61 pad 2: Net-(D21-A) -> Net-(D61-A)
- SW62 pad 1: Net-(U5-O6) -> Net-(U2-O6)
- SW62 pad 2: Net-(D35-A) -> Net-(D62-A)
- SW63 pad 1: Net-(U5-O6) -> Net-(U2-O6)
- SW63 pad 2: Net-(D49-A) -> Net-(D63-A)
- SW64 pad 1: Net-(U5-O6) -> Net-(U2-O6)
- SW64 pad 2: Net-(D63-A) -> Net-(D64-A)
- SW65 pad 1: Net-(U5-O6) -> Net-(U2-O6)
- SW65 pad 2: Net-(D51-A) -> Net-(D65-A)
- SW66 pad 1: Net-(U5-O6) -> Net-(U2-O6)
- SW66 pad 2: Net-(D52-A) -> Net-(D66-A)
- SW67 pad 1: Net-(U5-O6) -> Net-(U2-O6)
- SW67 pad 2: Net-(D53-A) -> Net-(D67-A)
- SW70 pad 1: Net-(U5-O7) -> Net-(U2-O7)
- SW71 pad 1: Net-(U5-O7) -> Net-(U2-O7)
- SW71 pad 2: Net-(D22-A) -> Net-(D71-A)
- SW72 pad 1: Net-(U5-O7) -> Net-(U2-O7)
- SW72 pad 2: Net-(D36-A) -> Net-(D72-A)
- SW73 pad 1: Net-(U5-O7) -> Net-(U2-O7)
- SW73 pad 2: Net-(D50-A) -> Net-(D73-A)
- SW74 pad 1: Net-(U5-O7) -> Net-(U2-O7)
- SW74 pad 2: Net-(D64-A) -> Net-(D74-A)
- SW75 pad 1: Net-(U5-O7) -> Net-(U2-O7)
- SW75 pad 2: Net-(D54-A) -> Net-(D75-A)
- SW76 pad 1: Net-(U5-O7) -> Net-(U2-O7)
- SW76 pad 2: Net-(D55-A) -> Net-(D76-A)
- SW77 pad 1: Net-(U5-O7) -> Net-(U2-O7)
- SW77 pad 2: Net-(D56-A) -> Net-(D77-A)
- U1 pad 1: /~{RD} -> /A1
- U1 pad 10: GND -> unconnected-(U1-O5-Pad10)
- U1 pad 12: GND -> /~{GPIO_E}
- U1 pad 13: GND -> /~{LCD_E}
- U1 pad 14: VCC -> /~{KB_E}
- U1 pad 2: /~{KB_E} -> /A2
- U1 pad 3: /~{KB_RD} -> /A3
- U1 pad 4: /~{KB_E} -> GND
- U1 pad 5: /~{WR} -> /~{IORQ}
- U1 pad 6: /~{KB_WR} -> VCC
- U1 pad 7: GND -> unconnected-(U1-O7-Pad7)
- U1 pad 8: unconnected-(U1-Pad8) -> GND
- U1 pad 9: GND -> unconnected-(U1-O6-Pad9)
- U2 pad 1: /~{LCD_E} -> GND
- U2 pad 10: unconnected-(U2-Pad10) -> GND
- U2 pad 11: GND -> /KB_WR
- U2 pad 12: unconnected-(U2-Pad12) -> Net-(U2-O4)
- U2 pad 13: GND -> /D4
- U2 pad 14: VCC -> /D5
- U2 pad 2: /LCD_E -> Net-(U2-O0)
- U2 pad 3: /~{KB_WR} -> /D0
- U2 pad 4: /KB_WR -> /D1
- U2 pad 5: /~{RD} -> Net-(U2-O1)
- U2 pad 6: /LCD_R/~{W} -> Net-(U2-O2)
- U2 pad 7: GND -> /D2
- U2 pad 8: unconnected-(U2-Pad8) -> /D3
- U2 pad 9: GND -> Net-(U2-O3)
- U4 pad 1: /A1 -> GND
- U4 pad 10: unconnected-(U4-O5-Pad10) -> GND
- U4 pad 11: unconnected-(U4-O4-Pad11) -> /GPIO_WR
- U4 pad 12: unconnected-(U4-O3-Pad12) -> Net-(J8-Pin_5)
- U4 pad 13: /~{LCD_E} -> /D4
- U4 pad 14: /~{KB_E} -> /D5
- U4 pad 15: /~{USB_IORQ} -> Net-(J8-Pin_6)
- U4 pad 16: VCC -> Net-(J8-Pin_7)
- U4 pad 2: /A2 -> Net-(J8-Pin_1)
- U4 pad 3: /A3 -> /D0
- U4 pad 4: GND -> /D1
- U4 pad 5: /~{IORQ} -> Net-(J8-Pin_2)
- U4 pad 6: VCC -> Net-(J8-Pin_3)
- U4 pad 7: unconnected-(U4-O7-Pad7) -> /D2
- U4 pad 8: GND -> /D3
- U4 pad 9: unconnected-(U4-O6-Pad9) -> Net-(J8-Pin_4)
- U5 pad 1: GND -> /~{GPIO_RD}
- U5 pad 11: /KB_WR -> Net-(J9-Pin_5)
- U5 pad 12: Net-(U5-O4) -> /D3
- U5 pad 13: /D4 -> Net-(J9-Pin_6)
- U5 pad 14: /D5 -> /D2
- U5 pad 15: Net-(U5-O5) -> Net-(J9-Pin_7)
- U5 pad 16: Net-(U5-O6) -> /D1
- U5 pad 17: /D6 -> Net-(J9-Pin_8)
- U5 pad 18: /D7 -> /D0
- U5 pad 19: Net-(U5-O7) -> /~{GPIO_RD}
- U5 pad 2: Net-(U5-O0) -> Net-(J9-Pin_1)
- U5 pad 3: /D0 -> /D7
- U5 pad 4: /D1 -> Net-(J9-Pin_2)
- U5 pad 5: Net-(U5-O1) -> /D6
- U5 pad 6: Net-(U5-O2) -> Net-(J9-Pin_3)
- U5 pad 7: /D2 -> /D5
- U5 pad 8: /D3 -> Net-(J9-Pin_4)
- U5 pad 9: Net-(U5-O3) -> /D4
- U6 pad 1: /~{KB_RD} -> /~{RD}
- U6 pad 10: GND -> /~{WR}
- U6 pad 11: Net-(D57-K) -> /~{GPIO_RD}
- U6 pad 12: /D3 -> /~{RD}
- U6 pad 13: Net-(D12-K) -> /~{GPIO_E}
- U6 pad 14: /D2 -> VCC
- U6 pad 2: Net-(D1-K) -> /~{KB_E}
- U6 pad 3: /D7 -> /~{KB_RD}
- U6 pad 4: Net-(D15-K) -> /~{KB_E}
- U6 pad 5: /D6 -> /~{WR}
- U6 pad 6: Net-(D29-K) -> /~{KB_WR}
- U6 pad 7: /D5 -> GND
- U6 pad 8: Net-(D43-K) -> Net-(U6-Pad8)
- U6 pad 9: /D4 -> /~{GPIO_E}
Other:
- board text removed: "PainfulDiodes BeanZee"

Commit message: Update BeanBoard.kicad_pcb
Parts:
- J5, J6: footprint Connector_PinSocket_2.54mm:PinSocket_1x07_P2.54mm_Vertical -> Connector_PinSocket_2.54mm:PinSocket_1x03_P2.54mm_Vertical
- moved J4 116.9 mm to (194.3, -32.6)
- moved RV1 100.1 mm to (203.5, -42.3)
- moved J3 87.0 mm to (267.4, -134.0)
- moved J6 85.2 mm to (198.9, -42.3)
- moved J5 85.2 mm to (194.3, -42.3)
- moved U1 82.6 mm to (264.1, -50.1)
- moved J2 10.8 mm to (250.5, -49.9)
- moved J9 10.8 mm to (259.7, -49.9)
- moved SW70 10.8 mm to (250.9, -187.2)
- moved SW72 10.8 mm to (250.9, -156.9)
- moved SW73 10.8 mm to (250.9, -141.7)
- moved SW74 10.8 mm to (250.9, -126.5)
- moved SW75 10.8 mm to (250.9, -111.4)
- moved SW76 10.8 mm to (250.9, -96.2)
- moved U6 10.8 mm to (250.3, -69.6)
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
Commit message: Update BeanBoard.kicad_pcb
Parts:
- moved J3 281.9 mm to (133.3, 114.0)
- moved J2 256.6 mm to (46.9, 106.4)
- moved J1 208.5 mm to (133.3, 108.9), turned to 180 degrees
- moved J6 202.3 mm to (100.2, 134.3), turned to 90 degrees
- moved J5 194.4 mm to (113.0, 134.3), turned to 90 degrees
- moved J4 180.0 mm to (46.9, 70.8)
- moved RV1 16.1 mm to (219.2, -38.8)
Other:
- board text added: "PainfulDiodes BeanZee"

Commit message: Update BeanBoard.kicad_pcb
Parts:
- moved SW60 307.5 mm to (-72.2, -198.7)
- moved SW61 289.7 mm to (-53.4, -198.7)
- moved C2 278.8 mm to (18.7, -31.9)
- moved C4 278.8 mm to (18.7, -23.8)
- moved C5 278.8 mm to (18.7, -19.8)
- moved C7 278.8 mm to (18.7, -11.7)
- moved C1 278.8 mm to (18.7, -36.0)
- moved C3 278.8 mm to (18.7, -27.9)
- moved C6 278.8 mm to (18.7, -15.7)
- moved J8 268.1 mm to (-2.67, 23.8)
- moved J9 268.1 mm to (1.93, 23.8)
- moved SW40 262.5 mm to (-57.4, -217.9)
- moved SW62 259.5 mm to (-21.0, -198.7)
- moved SW63 246.4 mm to (-4.67, -198.7)
- moved SW64 233.9 mm to (12.6, -198.7)
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
Commit message: Update BeanBoard.kicad_pcb
Parts:
- moved D00 266.9 mm to (-34.4, -272.3), turned to 90 degrees
- moved SW76 138.1 mm to (328.9, -197.6)
- moved SW77 138.1 mm to (348.6, -197.6)
- moved SW15 79.5 mm to (260.4, -257.5)
- moved SW16 79.5 mm to (278.6, -257.5)
- moved SW17 79.5 mm to (296.8, -257.5)
- moved SW36 73.4 mm to (277.9, -238.9)
- moved SW37 73.4 mm to (296.8, -238.9)
- moved SW35 73.4 mm to (259.4, -238.9)
- moved SW55 71.8 mm to (260.2, -218.0)
- moved SW56 71.8 mm to (279.4, -218.0)
- moved SW57 71.8 mm to (298.2, -218.0)
- moved SW00 58.8 mm to (-113.8, -257.9)
- moved SW20 58.8 mm to (-114.8, -237.7)
- moved SW40 58.8 mm to (-116.1, -217.8)
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