File: kicad/BeanBoard.kicad_pcb (KiCad board)
At the start: 2 copper layers, 161 parts, among them J1 BZ_Address, J2 BZ_Data, J3 BZ_Control, J4 BZ_Power, J5 BZ_IORQ_enable, J6 BZ_MREQ_enable, J7 LCD, J8 GPO, J9 GPI, SW00 SW_Push_45deg, SW01 SW_Push_45deg, SW02 SW_Push_45deg, SW03 SW_Push_45deg, SW04 SW_Push_45deg, SW05 SW_Push_45deg, SW06 SW_Push_45deg, SW07 SW_Push_45deg, SW10 SW_Push_45deg, SW11 SW_Push_45deg, SW12 SW_Push_45deg, SW13 SW_Push_45deg, SW14 SW_Push_45deg, SW15 SW_Push_45deg, SW16 SW_Push_45deg, SW17 SW_Push_45deg, SW20 SW_Push_45deg, SW21 SW_Push_45deg, SW22 SW_Push_45deg, SW23 SW_Push_45deg, SW24 SW_Push_45deg, SW25 SW_Push_45deg, SW26 SW_Push_45deg, SW27 SW_Push_45deg, SW30 SW_Push_45deg, SW31 SW_Push_45deg, SW32 SW_Push_45deg, SW33 SW_Push_45deg, SW34 SW_Push_45deg, SW35 SW_Push_45deg, SW36 SW_Push_45deg, SW37 SW_Push_45deg, SW40 SW_Push_45deg, SW41 SW_Push_45deg, SW42 SW_Push_45deg, SW43 SW_Push_45deg, SW44 SW_Push_45deg, SW45 SW_Push_45deg, SW46 SW_Push_45deg, SW47 SW_Push_45deg, SW50 SW_Push_45deg, SW51 SW_Push_45deg, SW52 SW_Push_45deg, SW53 SW_Push_45deg, SW54 SW_Push_45deg, SW55 SW_Push_45deg, SW56 SW_Push_45deg, SW57 SW_Push_45deg, SW60 SW_Push_45deg, SW61 SW_Push_45deg, SW62 SW_Push_45deg, SW63 SW_Push_45deg, SW64 SW_Push_45deg, SW65 SW_Push_45deg, SW66 SW_Push_45deg, SW67 SW_Push_45deg, SW70 SW_Push_45deg, SW71 SW_Push_45deg, SW72 SW_Push_45deg, SW73 SW_Push_45deg, SW74 SW_Push_45deg, SW75 SW_Push_45deg, SW76 SW_Push_45deg, SW77 SW_Push_45deg, U1 74LS138, U2 SN74LS373, U3 74LS244, U4 SN74LS373, U5 74LS244, U6 74LS32, U7 74LS04

Commit message: Update BeanBoard.kicad_pcb
Parts:
- moved SW55 319.1 mm to (-57.5, -186.8)
- moved SW56 319.0 mm to (-38.1, -186.8)
- moved SW57 318.8 mm to (-19.1, -186.8)
- moved SW76 264.8 mm to (64.5, -184.7)
- moved SW75 172.1 mm to (-0.04, -186.4)
- moved SW77 120.8 mm to (230.2, -221.2)
- moved SW17 86.2 mm to (230.2, -202.8)
- moved R1 70.9 mm to (322.1, -147.4)
- moved R2 70.9 mm to (322.1, -144.3)
- moved R4 70.9 mm to (322.1, -138.0)
- moved R5 70.9 mm to (322.1, -134.8)
- moved R6 70.9 mm to (322.1, -131.7)
- moved R7 70.9 mm to (322.1, -128.5)
- moved R9 70.9 mm to (322.1, -122.2)
- moved R8 70.9 mm to (322.1, -125.4)
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
Commit message: Update BeanBoard.kicad_pcb
Parts:
- moved D10 393.1 mm to (-180.3, -269.9), turned to 90 degrees
- moved D30 391.5 mm to (-180.3, -240.2), turned to 90 degrees
- moved D11 388.9 mm to (-172.5, -269.9), turned to 90 degrees
- moved D31 386.8 mm to (-172.5, -240.2), turned to 90 degrees
- moved D12 384.8 mm to (-164.6, -269.9), turned to 90 degrees
- moved D20 384.5 mm to (-180.3, -255.2), turned to 90 degrees
- moved D40 384.3 mm to (-180.3, -224.8), turned to 90 degrees
- moved D60 383.6 mm to (-180.3, -189.6), turned to 90 degrees
- moved D70 381.7 mm to (-180.3, -173.4), turned to 90 degrees
- moved D01 381.3 mm to (-172.5, -285.4), turned to 90 degrees
- moved D13 380.8 mm to (-156.8, -269.9), turned to 90 degrees
- moved D21 379.6 mm to (-172.5, -255.2), turned to 90 degrees
- moved D50 379.3 mm to (-180.3, -206.9), turned to 90 degrees
- moved D41 379.0 mm to (-172.5, -224.8), turned to 90 degrees
- moved D61 377.8 mm to (-172.5, -189.6), turned to 90 degrees
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
Commit message: Update BeanBoard.kicad_pcb
Parts:
- moved D36 411.2 mm to (276.0, -279.9)
- moved D37 411.2 mm to (283.8, -279.9)
- moved D15 357.1 mm to (215.5, -251.7)
- moved D35 356.6 mm to (215.4, -233.4)
- moved D34 345.4 mm to (196.4, -233.4)
- moved D14 336.6 mm to (187.2, -251.7)
- moved D33 334.2 mm to (177.4, -233.6)
- moved D13 325.4 mm to (168.1, -251.7)
- moved D32 323.1 mm to (158.4, -233.7)
- moved D12 314.2 mm to (149.0, -251.7)
- moved D31 311.7 mm to (139.2, -233.4)
- moved D11 303.0 mm to (130.0, -251.7)
- moved D30 300.5 mm to (120.2, -233.4)
- moved D10 291.8 mm to (110.9, -251.7)
- moved D27 227.6 mm to (101.1, -233.2)
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
Commit message: Update BeanBoard.kicad_pcb
Parts:
- moved D16 381.1 mm to (246.1, -233.1)
- moved D17 378.6 mm to (246.1, -196.7)
- moved D77 373.7 mm to (245.9, -214.7)
- moved D74 364.9 mm to (215.2, -196.0)
- moved D54 349.5 mm to (200.5, -214.4)
- moved D53 338.2 mm to (181.4, -214.4)
- moved D73 328.5 mm to (170.9, -196.5)
- moved D52 327.0 mm to (162.3, -214.4)
- moved D72 317.5 mm to (152.1, -196.5)
- moved D51 315.8 mm to (143.2, -214.4)
- moved D71 306.5 mm to (133.2, -196.5)
- moved D50 304.5 mm to (124.1, -214.4)
- moved D70 295.5 mm to (114.3, -196.5)
- moved D47 230.7 mm to (105.1, -215.0)
- moved D67 220.7 mm to (95.2, -196.5)
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
Commit message: Update BeanBoard.kicad_pcb
Parts:
- moved D00 448.4 mm to (83.7, 179.0)
- moved D01 448.4 mm to (102.7, 179.0)
- moved D02 448.4 mm to (121.8, 179.0)
- moved D03 448.4 mm to (140.8, 179.0)
- moved D04 448.4 mm to (159.9, 179.0)
- moved D05 448.4 mm to (178.9, 179.0)
- moved D06 448.4 mm to (198.0, 179.0)
- moved D07 448.4 mm to (217.1, 179.0)
- moved D10 448.4 mm to (236.1, 179.0)
- moved D11 448.4 mm to (255.2, 179.0)
- moved D12 448.4 mm to (274.2, 179.0)
- moved D13 448.4 mm to (293.3, 179.0)
- moved D14 448.4 mm to (312.3, 179.0)
- moved D15 448.4 mm to (340.7, 179.0)
- moved D16 448.4 mm to (371.2, 197.5)
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
Commit message: Update BeanBoard.kicad_pcb
Parts:
- moved J8 161.9 mm to (350.1, 117.7)
- moved J9 159.5 mm to (350.1, 86.1)
- moved R1 144.9 mm to (161.4, 113.6), turned to -90 degrees
- moved R2 140.7 mm to (164.6, 113.6), turned to -90 degrees
- moved R3 136.5 mm to (167.7, 113.6), turned to -90 degrees
- moved R4 132.3 mm to (170.9, 113.6), turned to -90 degrees
- moved R5 128.2 mm to (174.0, 113.6), turned to -90 degrees
- moved R6 124.1 mm to (177.2, 113.6), turned to -90 degrees
- moved U2 123.0 mm to (148.2, 130.7), turned to -90 degrees
- moved R7 120.0 mm to (180.3, 113.6), turned to -90 degrees
- moved R8 116.0 mm to (183.5, 113.6), turned to -90 degrees
- moved U3 115.0 mm to (180.4, 130.7), turned to -90 degrees
- moved U6 112.6 mm to (205.1, 130.7), turned to -90 degrees
- moved J7 110.8 mm to (235.8, 82.1)
- moved U1 105.1 mm to (232.3, 130.7), turned to -90 degrees
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Other:
- board outline added: 339.1 x 220.8 mm

Commit message: Update BeanBoard.kicad_pcb
Parts:
- moved J1 3.10 mm to (62.9, 131.7)
- moved J3 3.10 mm to (57.8, 131.7)
- moved J5 3.10 mm to (37.5, 111.4)
- moved J2 3.10 mm to (65.4, 45.4)
- moved J4 3.10 mm to (101.0, 45.4)
- moved J6 3.10 mm to (37.5, 98.7)
Other:
- board size 339.1 x 220.8 mm -> 339.1 x 217.6 mm
Changed lines of the file:
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@@
   (net 153 "unconnected-(U7-Pad12)")
   (footprint "Connector_PinSocket_2.54mm:PinSocket_1x16_P2.54mm_Vertical" (layer "F.Cu")
-    (at 62.89 128.64 90)
+    (at 62.89 131.74 90)
     (descr "Through hole straight socket strip, 1x16, 2.54mm pitch, single row (from Kicad 4.0.7), script generated")
     (tags "Through hole socket strip THT 1x16 2.54mm single row")
@@
   )
   (footprint "Connector_PinSocket_2.54mm:PinSocket_1x07_P2.54mm_Vertical" (layer "F.Cu")
-    (at 57.81 128.64 -90)
+    (at 57.81 131.74 -90)
     (descr "Through hole straight socket strip, 1x07, 2.54mm pitch, single row (from Kicad 4.0.7), script generated")
     (tags "Through hole socket strip THT 1x07 2.54mm single row")
@@
   )
   (footprint "Connector_PinSocket_2.54mm:PinSocket_1x03_P2.54mm_Vertical" (layer "F.Cu")
-    (at 37.49 108.32)
+    (at 37.49 111.42)
     (descr "Through hole straight socket strip, 1x03, 2.54mm pitch, single row (from Kicad 4.0.7), script generated")
     (tags "Through hole socket strip THT 1x03 2.54mm single row")
@@
   )
   (footprint "Connector_PinSocket_2.54mm:PinSocket_1x02_P2.54mm_Vertical" (layer "F.Cu")
-    (at 100.99 42.28 -90)
+    (at 100.99 45.38 -90)
     (descr "Through hole straight socket strip, 1x02, 2.54mm pitch, single row (from Kicad 4.0.7), script generated")
     (tags "Through hole socket strip THT 1x02 2.54mm single row")
@@
   )
   (footprint "Connector_PinSocket_2.54mm:PinSocket_1x03_P2.54mm_Vertical" (layer "F.Cu")
-    (at 37.49 95.62)
+    (at 37.49 98.72)
     (descr "Through hole straight socket strip, 1x03, 2.54mm pitch, single row (from Kicad 4.0.7), script generated")
     (tags "Through hole socket strip THT 1x03 2.54mm single row")
@@
   )
   (footprint "Connector_PinSocket_2.54mm:PinSocket_1x08_P2.54mm_Vertical" (layer "F.Cu")
-    (at 65.43 42.28 -90)
+    (at 65.43 45.38 -90)
     (descr "Through hole straight socket strip, 1x08, 2.54mm pitch, single row (from Kicad 4.0.7), script generated")
     (tags "Through hole socket strip THT 1x08 2.54mm single row")
@@
     (pad "4" thru_hole circle (at 12.5 5) (size 1.707896 1.707896) (drill 1.199896) (layers "*.Cu" "*.Mask"))
   )
-  (gr_rect (start 109.7 34.66) (end 29.87 138.26)
+  (gr_rect (start 109.7 37.76) (end 29.87 141.36)
     (stroke (width 0.1) (type default)) (fill none) (layer "F.SilkS"))
-  (gr_rect (start 20.670834 26.09) (end 359.800834 246.93)
+  (gr_rect (start 20.670834 29.37) (end 359.800834 246.93)
     (stroke (width 0.1) (type default)) (fill none) (layer "Edge.Cuts"))
-  (gr_text "PainfulDiodes\nBeanZee" (at 32.2 120.02 -90) (layer "F.SilkS")
+  (gr_text "PainfulDiodes\nBeanZee" (at 32.2 123.12 -90) (layer "F.SilkS")
     (effects (font (size 1.5 1.5) (thickness 0.1875)) (justify left bottom))
   )

Commit message: Update BeanBoard.kicad_pcb
Parts:
- moved D74 32.0 mm to (271.8, 214.5)
- moved SW74 32.0 mm to (256.2, 207.7)
- moved D37 27.9 mm to (331.4, 214.5)
- moved D16 27.6 mm to (313.1, 196.6)
- moved SW37 27.4 mm to (316.0, 207.7)
- moved J8 27.4 mm to (336.0, 94.2)
- moved J9 27.4 mm to (336.0, 62.6)
- moved D77 27.3 mm to (313.1, 214.5)
- moved SW16 27.1 mm to (297.6, 189.7)
- moved D17 27.0 mm to (313.0, 231.9)
- moved D36 26.9 mm to (294.7, 214.5)
- moved SW77 26.8 mm to (297.6, 207.7)
- moved SW17 26.5 mm to (297.6, 225.6)
- moved SW36 26.4 mm to (279.3, 207.7)
- moved D54 10.2 mm to (278.8, 196.6)
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Other:
- board size 339.1 x 217.6 mm -> 326.6 x 221.7 mm
