File: kicad/BeanBoard.kicad_pcb (KiCad board)
At the start: 2 copper layers, 326.6 x 221.7 mm, 161 parts, among them J1 BZ_Address, J2 BZ_Data, J3 BZ_Control, J4 BZ_Power, J5 BZ_IORQ_enable, J6 BZ_MREQ_enable, J7 LCD, J8 GPO, J9 GPI, SW00 SW_Push_45deg, SW01 SW_Push_45deg, SW02 SW_Push_45deg, SW03 SW_Push_45deg, SW04 SW_Push_45deg, SW05 SW_Push_45deg, SW06 SW_Push_45deg, SW07 SW_Push_45deg, SW10 SW_Push_45deg, SW11 SW_Push_45deg, SW12 SW_Push_45deg, SW13 SW_Push_45deg, SW14 SW_Push_45deg, SW15 SW_Push_45deg, SW16 SW_Push_45deg, SW17 SW_Push_45deg, SW20 SW_Push_45deg, SW21 SW_Push_45deg, SW22 SW_Push_45deg, SW23 SW_Push_45deg, SW24 SW_Push_45deg, SW25 SW_Push_45deg, SW26 SW_Push_45deg, SW27 SW_Push_45deg, SW30 SW_Push_45deg, SW31 SW_Push_45deg, SW32 SW_Push_45deg, SW33 SW_Push_45deg, SW34 SW_Push_45deg, SW35 SW_Push_45deg, SW36 SW_Push_45deg, SW37 SW_Push_45deg, SW40 SW_Push_45deg, SW41 SW_Push_45deg, SW42 SW_Push_45deg, SW43 SW_Push_45deg, SW44 SW_Push_45deg, SW45 SW_Push_45deg, SW46 SW_Push_45deg, SW47 SW_Push_45deg, SW50 SW_Push_45deg, SW51 SW_Push_45deg, SW52 SW_Push_45deg, SW53 SW_Push_45deg, SW54 SW_Push_45deg, SW55 SW_Push_45deg, SW56 SW_Push_45deg, SW57 SW_Push_45deg, SW60 SW_Push_45deg, SW61 SW_Push_45deg, SW62 SW_Push_45deg, SW63 SW_Push_45deg, SW64 SW_Push_45deg, SW65 SW_Push_45deg, SW66 SW_Push_45deg, SW67 SW_Push_45deg, SW70 SW_Push_45deg, SW71 SW_Push_45deg, SW72 SW_Push_45deg, SW73 SW_Push_45deg, SW74 SW_Push_45deg, SW75 SW_Push_45deg, SW76 SW_Push_45deg, SW77 SW_Push_45deg, U1 74LS138, U2 SN74LS373, U3 74LS244, U4 SN74LS373, U5 74LS244, U6 74LS32, U7 74LS04

Commit message: Update BeanBoard.kicad_pcb
Parts:
- moved J5 70.6 mm to (104.6, 133.5), turned to 90 degrees
- moved J3 69.6 mm to (124.9, 113.2), turned to 0 degrees
- moved J4 67.2 mm to (38.5, 70.0), turned to 0 degrees
- moved J1 66.3 mm to (124.9, 108.1), turned to 180 degrees
- moved J2 65.9 mm to (38.5, 105.6), turned to 0 degrees
- moved J6 64.6 mm to (91.9, 133.5), turned to 90 degrees
- moved C7 14.6 mm to (167.0, 133.3)
- moved U2 14.4 mm to (162.5, 130.7)
- moved C6 14.2 mm to (198.9, 133.4)
- moved U3 14.0 mm to (194.4, 130.7)
- moved C5 13.9 mm to (223.2, 133.2)
- moved U6 13.6 mm to (218.7, 130.7)
- moved C4 13.5 mm to (250.1, 133.2)
- moved U1 13.3 mm to (245.6, 130.7)
- moved C3 13.0 mm to (274.4, 133.3)
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Other:
- board size 326.6 x 221.7 mm -> 326.6 x 199.1 mm

Commit message: Update BeanBoard.kicad_pcb
Other:
- board text added: "' {dblquote}"
- board text added: ", <"
- board text added: "- _"
- board text added: ". >"
- board text added: "/ ?"
- board text added: "0 )"
- board text added: "1 !"
- board text added: "2 @"
- board text added: "3 #"
- board text added: "4 $"
- board text added: "5 %"
- board text added: "6 ^"
- board text added: "7 &"
- board text added: "8 *"
- board text added: "9 ("
- board text added: "; :"
- board text added: "= +"
- board text added: "A"
- board text added: "Alt"
- board text added: "B"
- board text added: "Back"
- board text added: "C"
- board text added: "Caps"
- board text added: "Cmd"
- board text added: "Ctrl"
- board text added: "D"
- board text added: "Down"
- board text added: "E"
- board text added: "Enter"
- board text added: "Esc"
- board text added: "F"
- board text added: "Fn"
- board text added: "G"
- board text added: "H"
- board text added: "I"
- board text added: "J"
- board text added: "K"
- board text added: "L"
- board text added: "Left"
- board text added: "M"
- board text added: "N"
- board text added: "O"
- board text added: "P"
- board text added: "Q"
- board text added: "R"
- board text added: "Right"
- board text added: "S"
- board text added: "Shift"
- board text added: "Space"
- board text added: "T"
- board text added: "Tab"
- board text added: "U"
- board text added: "Up"
- board text added: "V"
- board text added: "W"
- board text added: "X"
- board text added: "Y"
- board text added: "Z"
- board text added: "[ {"
- board text added: "\ |"
- board text added: "] }"
- board text added: "` ~"
Changed lines of the file:
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@@
   (gr_rect (start 18.850834 47.82) (end 345.410834 246.93)
     (stroke (width 0.1) (type default)) (fill none) (layer "Edge.Cuts"))
+  (gr_text "/ ?" (at 240.687321 202.493) (layer "F.SilkS")
+    (effects (font (size 2 2) (thickness 0.15)) (justify left bottom))
+  )
+  (gr_text "M" (at 186.494843 202.62) (layer "F.SilkS")
+    (effects (font (size 2 2) (thickness 0.15)) (justify left bottom))
+  )
+  (gr_text "Down" (at 299.92 220.403) (layer "F.SilkS")
+    (effects (font (size 2 2) (thickness 0.15)) (justify left bottom))
+  )
+  (gr_text "Shift" (at 33.65 202.493) (layer "F.SilkS")
+    (effects (font (size 2 2) (thickness 0.15)) (justify left bottom))
+  )
+  (gr_text "W" (at 81.12 166.927) (layer "F.SilkS")
+    (effects (font (size 2 2) (thickness 0.15)) (justify left bottom))
+  )
+  (gr_text "J" (at 176.37309 184.503) (layer "F.SilkS")
+    (effects (font (size 2 2) (thickness 0.15)) (justify left bottom))
+  )
+  (gr_text "I" (at 192.630005 166.8) (layer "F.SilkS")
+    (effects (font (size 2 2) (thickness 0.15)) (justify left bottom))
+  )
+  (gr_text "Left" (at 282.270682 202.493) (layer "F.SilkS")
+    (effects (font (size 2 2) (thickness 0.15)) (justify left bottom))
+  )
+  (gr_text "X" (at 93.762781 202.62) (layer "F.SilkS")
+    (effects (font (size 2 2) (thickness 0.15)) (justify left bottom))
+  )
+  (gr_text "D" (at 102.83209 184.63) (layer "F.SilkS")
+    (effects (font (size 2 2) (thickness 0.15)) (justify left bottom))
+  )
+  (gr_text "Fn" (at 35.35 220.033) (layer "F.SilkS")
+    (effects (font (size 2 2) (thickness 0.15)) (justify left bottom))
+  )
+  (gr_text "0 )" (at 217.567816 149.17) (layer "F.SilkS")
+    (effects (font (size 2 2) (thickness 0.15)) (justify left bottom))
+  )
+  (gr_text "V" (at 130.893343 202.493) (layer "F.SilkS")
+    (effects (font (size 2 2) (thickness 0.15)) (justify left bottom))
+  )
+  (gr_text "Y" (at 155.613407 166.673) (layer "F.SilkS")
+    (effects (font (size 2 2) (thickness 0.15)) (justify left bottom))
+  )
+  (gr_text "E" (at 100.27901 166.8) (layer "F.SilkS")
+    (effects (font (size 2 2) (thickness 0.15)) (justify left bottom))
+  )
+  (gr_text "Tab" (at 34.4 166.673) (layer "F.SilkS")
+    (effects (font (size 2 2) (thickness 0.15)) (justify left bottom))
+  )
+  (gr_text "F" (at 121.346045 184.503) (layer "F.SilkS")
+    (effects (font (size 2 2) (thickness 0.15)) (justify left bottom))
+  )
+  (gr_text "; :" (at 229.84009 184.63) (layer "F.SilkS")
+    (effects (font (size 2 2) (thickness 0.15)) (justify left bottom))
+  )
+  (gr_text "Space" (at 146.39 220.53) (layer "F.SilkS")
+    (effects (font (size 2 2) (thickness 0.15)) (justify left bottom))
+  )
+  (gr_text "Enter" (at 281.57 166.8) (layer "F.SilkS")
+    (effects (font (size 2 2) (thickness 0.15)) (justify left bottom))
+  )
+  (gr_text "7 &" (at 162.775385 149.297) (layer "F.SilkS")
+    (effects (font (size 2 2) (thickness 0.15)) (justify left bottom))
+  )
+  (gr_text ", <" (at 203.302759 202.62) (layer "F.SilkS")
+    (effects (font (size 2 2) (thickness 0.15)) (justify left bottom))
+  )
+  (gr_text "Alt" (at 73.018219 220.033) (layer "F.SilkS")
+    (effects (font (size 2 2) (thickness 0.15)) (justify left bottom))
+  )
+  (gr_text "6 ^" (at 144.468908 149.043) (layer "F.SilkS")
+    (effects (font (size 2 2) (thickness 0.15)) (justify left bottom))
+  )
+  (gr_text "5 %" (at 126.289431 149.17) (layer "F.SilkS")
+    (effects (font (size 2 2) (thickness 0.15)) (justify left bottom))
+  )
+  (gr_text "C" (at 112.264562 202.493) (layer "F.SilkS")
+    (effects (font (size 2 2) (thickness 0.15)) (justify left bottom))
+  )
+  (gr_text "9 (" (at 199.388339 149.043) (layer "F.SilkS")
+    (effects (font (size 2 2) (thickness 0.15)) (justify left bottom))
+  )
+  (gr_text ". >" (at 222.18554 202.62) (layer "F.SilkS")
+    (effects (font (size 2 2) (thickness 0.15)) (justify left bottom))
+  )
+  (gr_text "[ {" (at 246.562201 166.8) (layer "F.SilkS")
+    (effects (font (size 2 2) (thickness 0.15)) (justify left bottom))
+  )
+  (gr_text "Up" (at 302.05 184.63) (layer "F.SilkS")
+    (effects (font (size 2 2) (thickness 0.15)) (justify left bottom))
+  )
+  (gr_text "R" (at 118.850809 166.8) (layer "F.SilkS")
+    (effects (font (size 2 2) (thickness 0.15)) (justify left bottom))
+  )
+  (gr_text "= +" (at 254.18077 149.17) (layer "F.SilkS")
+    (effects (font (size 2 2) (thickness 0.15)) (justify left bottom))
+  )
+  (gr_text "3 #" (at 89.422477 149.17) (layer "F.SilkS")
+    (effects (font (size 2 2) (thickness 0.15)) (justify left bottom))
+  )
+  (gr_text "Z" (at 74.88 202.62) (layer "F.SilkS")
+    (effects (font (size 2 2) (thickness 0.15)) (justify left bottom))
+  )
+  (gr_text "L" (at 213.02 184.63) (layer "F.SilkS")
+    (effects (font (size 2 2) (thickness 0.15)) (justify left bottom))
+  )
+  (gr_text "4 $" (at 107.982954 149.17) (layer "F.SilkS")
+    (effects (font (size 2 2) (thickness 0.15)) (justify left bottom))
+  )
+  (gr_text "H" (at 157.986135 184.503) (layer "F.SilkS")
+    (effects (font (size 2 2) (thickness 0.15)) (justify left bottom))
+  )
+  (gr_text "P" (at 229.519603 166.8) (layer "F.SilkS")
+    (effects (font (size 2 2) (thickness 0.15)) (justify left bottom))
+  )
   (gr_text "PainfulDiodes\nBeanZee" (at 116.26 138.81) (layer "F.SilkS")
     (effects (font (size 1.5 1.5) (thickness 0.1875)) (justify left bottom))
   )
+  (gr_text "T" (at 137.041608 166.8) (layer "F.SilkS")
+    (effects (font (size 2 2) (thickness 0.15)) (justify left bottom))
+  )
+  (gr_text "S" (at 84.572135 184.503) (layer "F.SilkS")
+    (effects (font (size 2 2) (thickness 0.15)) (justify left bottom))
+  )
+  (gr_text "G" (at 139.86 184.63) (layer "F.SilkS")
+    (effects (font (size 2 2) (thickness 0.15)) (justify left bottom))
+  )
+  (gr_text "Back" (at 281.93 149.17) (layer "F.SilkS")
+    (effects (font (size 2 2) (thickness 0.15)) (justify left bottom))
+  )
+  (gr_text "B" (at 149.522124 202.493) (layer "F.SilkS")
+    (effects (font (size 2 2) (thickness 0.15)) (justify left bottom))
+  )
+  (gr_text "Caps" (at 33.65 184.503) (layer "F.SilkS")
+    (effects (font (size 2 2) (thickness 0.15)) (justify left bottom))
+  )
+  (gr_text "Right" (at 318.12 202.493) (layer "F.SilkS")
+    (effects (font (size 2 2) (thickness 0.15)) (justify left bottom))
+  )
+  (gr_text "N" (at 167.993062 202.493) (layer "F.SilkS")
+    (effects (font (size 2 2) (thickness 0.15)) (justify left bottom))
+  )
+  (gr_text "Q" (at 62.675201 166.927) (layer "F.SilkS")
+    (effects (font (size 2 2) (thickness 0.15)) (justify left bottom))
+  )
+  (gr_text "\\ |" (at 266.36 184.63) (layer "F.SilkS")
+    (effects (font (size 2 2) (thickness 0.15)) (justify left bottom))
+  )
+  (gr_text "K" (at 194.887045 184.63) (layer "F.SilkS")
+    (effects (font (size 2 2) (thickness 0.15)) (justify left bottom))
+  )
+  (gr_text "Ctrl" (at 54.389438 220.033) (layer "F.SilkS")
+    (effects (font (size 2 2) (thickness 0.15)) (justify left bottom))
+  )
+  (gr_text "1 !" (at 53.063523 149.17) (layer "F.SilkS")
+    (effects (font (size 2 2) (thickness 0.15)) (justify left bottom))
+  )
+  (gr_text "Cmd" (at 91.52 220.53) (layer "F.SilkS")
+    (effects (font (size 2 2) (thickness 0.15)) (justify left bottom))
+  )
+  (gr_text "O" (at 210.820804 166.8) (layer "F.SilkS")
+    (effects (font (size 2 2) (thickness 0.15)) (justify left bottom))
+  )
+  (gr_text "U" (at 173.931206 166.8) (layer "F.SilkS")
+    (effects (font (size 2 2) (thickness 0.15)) (justify left bottom))
+  )
+  (gr_text "Esc" (at 34.66 149.17) (layer "F.SilkS")
+    (effects (font (size 2 2) (thickness 0.15)) (justify left bottom))
+  )
+  (gr_text "`  ~" (at 54.55 202.62) (layer "F.SilkS")
+    (effects (font (size 2 2) (thickness 0.15)) (justify left bottom))
+  )
+  (gr_text "' {dblquote}" (at 248.100045 184.503) (layer "F.SilkS")
+    (effects (font (size 2 2) (thickness 0.15)) (justify left bottom))
+  )
+  (gr_text "2 @" (at 71.37 149.17) (layer "F.SilkS")
+    (effects (font (size 2 2) (thickness 0.15)) (justify left bottom))
+  )
+  (gr_text "A" (at 66.18518 184.503) (layer "F.SilkS")
+    (effects (font (size 2 2) (thickness 0.15)) (justify left bottom))
+  )
+  (gr_text "8 *" (at 180.954862 149.17) (layer "F.SilkS")
+    (effects (font (size 2 2) (thickness 0.15)) (justify left bottom))
+  )
+  (gr_text "] }" (at 264.88 166.673) (layer "F.SilkS")
+    (effects (font (size 2 2) (thickness 0.15)) (justify left bottom))
+  )
+  (gr_text "Shift" (at 259.325607 202.62) (layer "F.SilkS")
+    (effects (font (size 2 2) (thickness 0.15)) (justify left bottom))
+  )
+  (gr_text "- _" (at 236.001293 149.043) (layer "F.SilkS")
+    (effects (font (size 2 2) (thickness 0.15)) (justify left bottom))
+  )
   (group "" (id 1f489ed8-efd6-4aa2-8e73-cfa8a5897d33)

Commit message: Update BeanBoard.kicad_pcb
Parts:
- added J10: Power, Connector_PinSocket_2.54mm:PinSocket_1x02_P2.54mm_Vertical, F.Cu at (349.8, 51.9)
- moved U2 176.8 mm to (336.8, 101.1)
- moved C7 175.8 mm to (340.3, 103.6)
- moved U3 149.6 mm to (336.8, 84.7)
- moved C6 148.8 mm to (340.3, 87.1)
- moved R2 110.6 mm to (286.5, 101.2)
- moved R3 110.6 mm to (289.6, 101.2)
- moved R5 110.6 mm to (295.9, 101.2)
- moved R7 110.6 mm to (302.2, 101.2)
- moved R8 110.6 mm to (305.4, 101.2)
- moved R1 110.6 mm to (283.3, 101.2)
- moved R4 110.6 mm to (292.8, 101.2)
- moved R6 110.6 mm to (299.1, 101.2)
- moved U6 94.5 mm to (301.3, 84.7)
- moved C5 93.6 mm to (304.7, 87.3)
- moved U7 84.9 mm to (301.3, 51.7)
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Other:
- board text added: "PainfulDiodes BeanBoard"

Commit message: Update BeanBoard.kicad_pcb
Routing:
- net Net-(D06-K): track 0.00 -> 204.8 mm
- net Net-(D05-K): track 0.00 -> 189.7 mm
- net Net-(U2-O1): track 0.00 -> 156.4 mm
- net Net-(U2-O4): track 0.00 -> 147.3 mm
- net Net-(U2-O2): track 0.00 -> 144.5 mm
- net Net-(U2-O6): track 0.00 -> 139.0 mm
- net Net-(U2-O3): track 0.00 -> 137.1 mm
- net Net-(U2-O0): track 0.00 -> 135.5 mm
- net Net-(D04-K): track 0.00 -> 126.8 mm
- net Net-(D01-K): track 0.00 -> 126.4 mm
- net Net-(D02-K): track 0.00 -> 126.4 mm
- net Net-(D03-K): track 0.00 -> 126.4 mm
- net Net-(U2-O7): track 0.00 -> 120.9 mm
- net Net-(D00-K): track 0.00 -> 119.5 mm
- net Net-(U2-O5): track 0.00 -> 118.4 mm
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
Commit message: Update BeanBoard.kicad_pcb
Routing:
- net Net-(D07-K): track 63.2 -> 467.9 mm, vias 0 -> 1
- net Net-(D00-K): track 119.5 -> 521.5 mm
- net Net-(U2-O6): track 139.0 -> 499.1 mm
- net Net-(U2-O4): track 147.3 -> 485.6 mm, vias 0 -> 1
- net Net-(U2-O2): track 144.5 -> 479.9 mm, vias 0 -> 1
- net Net-(D01-K): track 126.4 -> 374.6 mm, vias 0 -> 2
- net Net-(U2-O5): track 118.4 -> 360.2 mm, vias 0 -> 1
- net Net-(U2-O7): track 120.9 -> 325.2 mm
- net Net-(U2-O0): track 135.5 -> 322.2 mm
- net Net-(D05-K): track 189.7 -> 348.2 mm
- net Net-(D03-K): track 126.4 -> 278.5 mm
- net Net-(D02-K): track 126.4 -> 276.1 mm
- net Net-(D04-K): track 126.8 -> 276.4 mm
- net Net-(D06-K): track 204.8 -> 346.7 mm
- net Net-(U2-O3): track 137.1 -> 250.1 mm, vias 0 -> 2
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
Commit message: Update BeanBoard.kicad_pcb
Parts:
- moved R1 146.4 mm to (388.8, -0.32)
- moved R3 146.4 mm to (395.1, -0.32)
- moved R4 146.4 mm to (398.3, -0.32)
- moved R5 146.4 mm to (401.4, -0.32)
- moved R6 146.4 mm to (404.6, -0.32)
- moved R8 146.4 mm to (410.9, -0.32)
- moved R2 146.4 mm to (392.0, -0.32)
- moved R7 146.4 mm to (407.7, -0.32)
- moved R9 126.7 mm to (324.4, -5.67)
- moved RV1 126.7 mm to (309.8, -3.81)
Routing:
- net Net-(D06-K): track 346.7 -> 468.0 mm, vias 0 -> 2
- net Net-(D02-K): track 276.1 -> 394.1 mm, vias 0 -> 1
- net Net-(D03-K): track 278.5 -> 371.6 mm, vias 0 -> 1
- net Net-(D04-K): track 276.4 -> 352.2 mm, vias 0 -> 1
- net Net-(D05-K): track 348.2 -> 420.5 mm, vias 0 -> 1
- net Net-(D01-K): track 374.6 -> 434.6 mm, vias 2 -> 3
- net Net-(U2-O1): track 253.1 -> 258.5 mm, vias 0 -> 1
- net Net-(U2-O3): track 250.1 -> 255.4 mm
- net Net-(U2-O2): track 479.9 -> 484.1 mm
- net Net-(D56-A): track 0.00 -> 3.64 mm
- net Net-(D07-K): track 467.9 -> 471.5 mm, vias 1 -> 2
- net Net-(D17-A): track 0.00 -> 3.44 mm
- net Net-(U2-O6): track 499.1 -> 502.4 mm
- net Net-(U2-O5): track 360.2 -> 363.2 mm
- net Net-(U2-O4): track 485.6 -> 488.3 mm
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
Commit message: Update BeanBoard.kicad_pcb
Parts:
- moved R7 147.9 mm to (286.6, 84.6)
- moved R8 136.4 mm to (304.2, 84.6)
- moved R5 135.8 mm to (295.4, 84.6)
- moved R6 133.7 mm to (301.3, 84.6)
- moved R3 133.2 mm to (292.5, 84.6)
- moved R2 133.0 mm to (289.6, 84.6)
- moved R4 131.1 mm to (298.4, 84.6)
- moved R1 117.8 mm to (307.2, 84.6)
- moved U6 20.3 mm to (298.7, 104.8)
- moved C5 20.1 mm to (302.1, 107.2)
- moved C3 2.56 mm to (302.3, 54.1)
- moved U7 2.55 mm to (298.7, 51.7)
Routing:
- net /D0: track 0.00 -> 356.9 mm
- net /D1: track 0.00 -> 355.9 mm, vias 0 -> 2
- net /D3: track 0.00 -> 350.5 mm, vias 0 -> 4
- net /D2: track 0.00 -> 347.5 mm, vias 0 -> 2
- net /D7: track 0.00 -> 341.6 mm, vias 0 -> 1
- net /D6: track 0.00 -> 337.9 mm, vias 0 -> 2
- net /D5: track 0.00 -> 331.2 mm, vias 0 -> 1
- net /D4: track 0.00 -> 328.8 mm, vias 0 -> 1
- net Net-(D00-K): track 524.0 -> 557.2 mm
- net Net-(D06-K): track 468.0 -> 497.5 mm, vias 2 -> 3
- net Net-(D07-K): track 471.5 -> 497.8 mm
- net Net-(D01-K): track 434.6 -> 460.7 mm, vias 3 -> 4
- net Net-(D02-K): track 394.1 -> 418.4 mm, vias 1 -> 2
- net Net-(D04-K): track 352.2 -> 372.8 mm, vias 1 -> 2
- net GND: track 0.00 -> 20.5 mm
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
Commit message: Update BeanBoard.kicad_pcb
Routing:
- net /~{USB_IORQ}: track 0.00 -> 198.2 mm, vias 0 -> 1
- net /A1: track 0.00 -> 173.0 mm, vias 0 -> 3
- net /~{IORQ}: track 0.00 -> 171.5 mm, vias 0 -> 1
- net /A2: track 0.00 -> 170.6 mm, vias 0 -> 3
- net /~{RD}: track 0.00 -> 170.2 mm
- net /A3: track 0.00 -> 166.1 mm, vias 0 -> 3
- net /LCD_E: track 0.00 -> 113.8 mm, vias 0 -> 2
- net /RD: track 0.00 -> 104.5 mm, vias 0 -> 1
- net /KB_WR: track 0.00 -> 99.0 mm
- net /~{KB_WR}: track 0.00 -> 65.5 mm
- net /D4: track 328.8 -> 393.9 mm, vias 1 -> 2
- net Net-(U6-Pad8): track 0.00 -> 60.4 mm, vias 0 -> 1
- net /D5: track 331.2 -> 385.1 mm, vias 1 -> 3
- net /GPIO_WR: track 0.00 -> 52.8 mm
- net /D6: track 337.9 -> 382.9 mm, vias 2 -> 3
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